File: Hardware/Controller base/Controller base.kicad_pcb (KiCad board)
At the start: 2 copper layers, 63.2 x 68.6 mm, 35 parts, among them J1 USB_C_Receptacle_USB2.0_16P, J2 Conn_01x05_Pin, J3 right face mod, J4 left face mod, J5 left sholder, J6 right sholder, SW1 SW_Push, SW2 SW_Push, SW3 SW_Push, SW4 SW_Push, U1 AZ1117CH-3.3TRG1, U2 ESP32-S3-WROOM-1U-N4

Commit message: update
Parts:
- J2: moved to B.Cu
- moved J2 60.5 mm to (131.1, 134.1)
- moved D4 24.4 mm to (143.1, 116.7)
- moved D5 24.4 mm to (146.2, 116.7)
- moved D6 24.4 mm to (149.4, 116.7)
- moved D7 24.4 mm to (152.3, 116.7)
- moved C8 8.11 mm to (136.2, 107.0), turned to 180 degrees
- moved R4 8.03 mm to (135.2, 103.4), turned to -90 degrees
- moved C1 5.33 mm to (139.8, 88.8), turned to 180 degrees
- moved C2 3.69 mm to (139.7, 91.7), turned to 180 degrees
Connections:
- J2 pad 4: GPIO41 -> GPIO42
- J2 pad 5: GPIO42 -> GPIO41
Routing:
- added copper zone on F.Cu, net GND
Other:
- board size 63.2 x 68.6 mm -> 63.2 x 68.5 mm

Commit message: update pcb
Parts:
- C3: footprint Capacitor_SMD:C_0805_2012Metric_Pad1.18x1.45mm_HandSolder -> Capacitor_SMD:C_0603_1608Metric_Pad1.08x0.95mm_HandSolder
- U1: moved to B.Cu
- moved R3 26.1 mm to (131.7, 110.4)
- moved R10 20.8 mm to (150.0, 111.8), turned to 180 degrees
- moved R9 18.3 mm to (150.0, 114.0), turned to 180 degrees
- moved R8 16.2 mm to (150.0, 116.2), turned to 180 degrees
- moved R7 14.8 mm to (150.0, 118.4), turned to 180 degrees
- moved D7 13.2 mm to (139.8, 121.0), turned to 90 degrees
- moved U1 10.4 mm to (147.6, 96.2)
- moved D6 8.29 mm to (142.4, 121.0), turned to 90 degrees
- moved J3 7.20 mm to (164.8, 117.7)
- moved D4 5.94 mm to (147.1, 121.0), turned to 90 degrees
- moved R6 5.52 mm to (135.5, 99.0)
- moved J4 5.35 mm to (122.6, 123.1)
- moved C3 4.74 mm to (154.5, 131.0)
- moved D5 4.55 mm to (144.8, 121.0), turned to 90 degrees
- moved R4 4.43 mm to (139.5, 104.4), turned to 180 degrees
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Routing:
- net GND: track 0.00 -> 70.8 mm, vias 0 -> 3
- net D+: track 0.00 -> 35.6 mm
- net D-: track 0.00 -> 35.3 mm
- net VBUS: track 0.00 -> 17.9 mm
- net Net-(D7-A): track 0.00 -> 13.7 mm
- net ESP_3.3V: track 0.00 -> 12.7 mm
- net VCC_5V: track 0.00 -> 10.9 mm
- net VCC_3V3: track 0.00 -> 10.3 mm
- net Net-(D6-A): track 0.00 -> 9.94 mm
- net TXD0: track 0.00 -> 9.70 mm
- net RXD0: track 0.00 -> 9.28 mm
- net GPIO42: track 0.00 -> 6.65 mm
- net Net-(D5-A): track 0.00 -> 6.44 mm
- net GPIO41: track 0.00 -> 6.16 mm
- net GPIO0: track 0.00 -> 5.28 mm
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