File: Hardware/Controller base V0.5/Input Modules.kicad_sch (KiCad schematic)
At the start: 0 parts

Commit message: update
Parts:
- added J3: right face mod, Connector_PinHeader_1.27mm:PinHeader_2x07_P1.27mm_Vertical, symbol Connector_Generic:Conn_02x07_Odd_Even
- added J4: left face mod, Connector_PinHeader_1.27mm:PinHeader_2x07_P1.27mm_Vertical, symbol Connector_Generic:Conn_02x07_Odd_Even
- added J5: left sholder, Connector_PinHeader_1.27mm:PinHeader_1x04_P1.27mm_Vertical, symbol Library:Conn_01x04_Pin
- added J6: right sholder, Connector_PinHeader_1.27mm:PinHeader_1x04_P1.27mm_Vertical, symbol Library:Conn_01x04_Pin
Connections:
- new net GND: J3.13 (Pin_13), J3.5 (Pin_5), J4.14 (Pin_14), J4.6 (Pin_6), J5.4 (Pin_4), J6.4 (Pin_4)
- new net GPIO1: J3.14 (Pin_14)
- new net GPIO10: J3.8 (Pin_8)
- new net GPIO11: J4.13 (Pin_13)
- new net GPIO12: J4.9 (Pin_9)
- new net GPIO13: J4.7 (Pin_7)
- new net GPIO14: J4.11 (Pin_11)
- new net GPIO15: J3.10 (Pin_10)
- new net GPIO16: J4.1 (Pin_1)
- new net GPIO17: J6.2 (Pin_2)
- new net GPIO18: J5.2 (Pin_2)
- new net GPIO2: J3.12 (Pin_12)
- new net GPIO3: J6.3 (Pin_3)
- new net GPIO4: J4.5 (Pin_5)
- new net GPIO5: J4.3 (Pin_3)
- new net GPIO6: J5.3 (Pin_3)
- new net GPIO7: J3.2 (Pin_2)
- new net GPIO8: J3.4 (Pin_4)
- new net GPIO9: J3.6 (Pin_6)
- new net VCC_3V3: J3.1 (Pin_1), J3.9 (Pin_9), J4.10 (Pin_10), J4.2 (Pin_2), J5.1 (Pin_1), J6.1 (Pin_1)
- no-connect marks 0 -> 6
