File: Hardware/Controller base V0.6/Input Modules.kicad_sch (KiCad schematic)
At the start: 4 parts, among them J3 right face mod, J4 left face mod, J5 left sholder, J6 right sholder

Commit message: updated carrier board
Other:
- company: (none) -> OSHE
Changed lines of the file:
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@@
 	(generator_version "9.0")
 	(paper "A4")
+	(title_block
+		(date "2025-09-26")
+		(rev "0.6")
+		(company "OSHE")
+	)
 	(junction
 		(at 36.83 71.12)

Commit message: updated liby used
Parts:
- J3, J4: symbol Connector_Generic:Conn_02x07_Odd_Even -> MCU_Controller:Conn_02x07_Odd_Even; now left out of the parts list
- J5, J6: symbol Library:Conn_01x04_Pin -> MCU_Controller:Conn_01x04_Pin; now left out of the parts list
Changed lines of the file:
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@@
 	)
 	(symbol
-		(lib_id "Library:+3V3")
+		(lib_id "MCU_Controller:+3V3")
 		(at 36.83 34.29 0)
 		(unit 1)
@@
 	)
 	(symbol
-		(lib_id "Connector_Generic:Conn_02x07_Odd_Even")
+		(lib_id "MCU_Controller:Conn_02x07_Odd_Even")
 		(at 52.07 102.87 0)
 		(unit 1)
 		(exclude_from_sim no)
-		(in_bom yes)
+		(in_bom no)
 		(on_board no)
 		(dnp no)
@@
 	)
 	(symbol
-		(lib_id "Library:Conn_01x04_Pin")
+		(lib_id "MCU_Controller:Conn_01x04_Pin")
 		(at 62.23 41.91 0)
 		(mirror y)
 		(unit 1)
 		(exclude_from_sim no)
-		(in_bom yes)
+		(in_bom no)
 		(on_board no)
 		(dnp no)
@@
 	)
 	(symbol
-		(lib_id "Library:Conn_01x04_Pin")
+		(lib_id "MCU_Controller:Conn_01x04_Pin")
 		(at 62.23 57.15 0)
 		(mirror y)
 		(unit 1)
 		(exclude_from_sim no)
-		(in_bom yes)
+		(in_bom no)
 		(on_board no)
 		(dnp no)
@@
 	)
 	(symbol
-		(lib_id "Library:GND")
+		(lib_id "MCU_Controller:GND")
 		(at 30.48 36.83 180)
 		(unit 1)
@@
 	)
 	(symbol
-		(lib_id "Connector_Generic:Conn_02x07_Odd_Even")
+		(lib_id "MCU_Controller:Conn_02x07_Odd_Even")
 		(at 54.61 78.74 0)
 		(mirror y)
 		(unit 1)
 		(exclude_from_sim no)
-		(in_bom yes)
+		(in_bom no)
 		(on_board no)
 		(dnp no)
