File: Hardware/Controller base V0.6/Controller base V0.6.kicad_sch (KiCad schematic)
At the start: 35 parts, among them J1 USB_C_Receptacle_USB2.0_16P, J2 Conn_01x05_Pin, J7 Conn_02x10_Counter_Clockwise, J8 Conn_02x10_Counter_Clockwise, SW1 SW_Push, SW2 SW_Push, SW3 SW_Push, SW4 SW_Push, U1 AZ1117CH-3.3TRG1, U2 ESP32-S3-WROOM-1U-N4

Commit message: .6 done
Parts:
- R1, R2: footprint Resistor_SMD:R_0805_2012Metric_Pad1.20x1.40mm_HandSolder -> Resistor_SMD:R_0603_1608Metric_Pad0.98x0.95mm_HandSolder
Changed lines of the file:
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@@
 			)
 		)
-		(property "Footprint" "Resistor_SMD:R_0805_2012Metric_Pad1.20x1.40mm_HandSolder"
+		(property "Footprint" "Resistor_SMD:R_0603_1608Metric_Pad0.98x0.95mm_HandSolder"
 			(at 45.72 86.868 90)
 			(effects
@@
 			)
 		)
-		(property "Footprint" "Resistor_SMD:R_0805_2012Metric_Pad1.20x1.40mm_HandSolder"
+		(property "Footprint" "Resistor_SMD:R_0603_1608Metric_Pad0.98x0.95mm_HandSolder"
 			(at 45.72 81.788 90)
 			(effects
@@
 		)
 		(instances
-			(project "Controller base V0.5"
+			(project "Controller base V0.6"
 				(path "/5ff5287b-60c7-4258-8bdb-42f045207b2d"
 					(page "2")

Commit message: updated carrier board
Parts:
- D2: symbol Library:PRTR5V0U2X_215 -> PRTR5V0U2X_215:PRTR5V0U2X_215
- J7, J8: footprint Connector_Hirose_DF40:Hirose_DF40C-20DS-0.4V_2x10_P0.4mm -> DF40C:HRS_DF40C-20DP-0.4V_51_; symbol Connector_Generic:Conn_02x10_Odd_Even -> DF40C:DF40C-20DP-0.4V_51_; MANUFACTURER (none) -> Hirose Electric; MAXIMUM_PACKAGE_HEIGHT (none) -> 1.29mm; PARTREV (none) -> 02/2020; STANDARD (none) -> Manufacturer Recommendations
- SW4: footprint Button_Switch_SMD:SW_SPST_PTS647_Sx38 -> Button_Switch_SMD:SW_Push_1P1T_XKB_TS-1187A
Connections:
- net GND: now also J7.12, J7.14, J7.16, J8.16, J8.18, J8.20; no longer J7.11 (Pin_11), J7.13 (Pin_13), J7.15 (Pin_15), J8.15 (Pin_15), J8.17 (Pin_17), J8.19 (Pin_19)
- net GPIO1: now also J8.11; no longer J8.12 (Pin_12)
- net GPIO10: now also J7.11; no longer J7.12 (Pin_12)
- net GPIO11: now also J7.9; no longer J7.10 (Pin_10)
- net GPIO12: now also J7.7; no longer J7.8 (Pin_8)
- net GPIO13: now also J7.5; no longer J7.6 (Pin_6)
- net GPIO14: now also J7.3; no longer J7.4 (Pin_4)
- net GPIO15: now also J8.10; no longer J8.9 (Pin_9)
- net GPIO16: now also J8.12; no longer J8.11 (Pin_11)
- net GPIO17: now also J8.14; no longer J8.13 (Pin_13)
- net GPIO18: now also J7.19; no longer J7.20 (Pin_20)
- net GPIO2: now also J8.9; no longer J8.10 (Pin_10)
- net GPIO21: now also J7.1; no longer J7.2 (Pin_2)
- net GPIO3: now also J7.15; no longer J7.16 (Pin_16)
- net GPIO35: now also J8.2; no longer J8.1 (Pin_1)
- net GPIO36: now also J8.4; no longer J8.3 (Pin_3)
- net GPIO37: now also J8.6; no longer J8.5 (Pin_5)
- net GPIO38: now also J8.8; no longer J8.7 (Pin_7)
- net GPIO4: now also J8.13; no longer J8.14 (Pin_14)
- net GPIO41: now also J8.1; no longer J8.2 (Pin_2)
- net GPIO42: now also J8.3; no longer J8.4 (Pin_4)
- net GPIO47: now also J7.4; no longer J7.3 (Pin_3)
- net GPIO48: now also J7.2; no longer J7.1 (Pin_1)
- net GPIO5: now also J8.15; no longer J8.16 (Pin_16)
- net GPIO6: now also J8.17; no longer J8.18 (Pin_18)
- net GPIO7: now also J8.19; no longer J8.20 (Pin_20)
- net GPIO8: now also J7.17; no longer J7.18 (Pin_18)
- net GPIO9: now also J7.13; no longer J7.14 (Pin_14)
- net RXD0: now also J8.5; no longer J8.6 (Pin_6)
- net TXD0: now also J8.7; no longer J8.8 (Pin_8)
- net VCC_3V3: now also J7.10, J7.6, J7.8; no longer J7.5 (Pin_5), J7.7 (Pin_7), J7.9 (Pin_9)
- net VCC_5V: now also J7.18, J7.20; no longer J7.17 (Pin_17), J7.19 (Pin_19)
Other:
- company: (none) -> OSHE
- title: (none) -> MCU Carrier Board
Changed lines of the file:
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@@
 	(generator_version "9.0")
 	(paper "A4")
+	(title_block
+		(title "MCU Carrier Board")
+		(date "2025-09-26")
+		(rev "0.6")
+		(company "OSHE")
+	)
 	(rectangle
 		(start 12.7 144.78)
@@
 	(wire
 		(pts
-			(xy 264.16 52.07) (xy 271.78 52.07)
+			(xy 265.43 83.82) (xy 271.78 83.82)
 		)
 		(stroke
@@
 	(wire
 		(pts
-			(xy 34.29 80.01) (xy 34.29 77.47)
+			(xy 264.16 52.07) (xy 271.78 52.07)
 		)
 		(stroke
@@
 	(wire
 		(pts
-			(xy 144.78 41.91) (xy 144.78 44.45)
+			(xy 34.29 80.01) (xy 34.29 77.47)
 		)
 		(stroke
@@
 	(wire
 		(pts
-			(xy 49.53 176.53) (xy 58.42 176.53)
+			(xy 144.78 41.91) (xy 144.78 44.45)
 		)
 		(stroke
@@
 	(wire
 		(pts
-			(xy 102.87 33.02) (xy 102.87 31.75)
+			(xy 49.53 176.53) (xy 58.42 176.53)
 		)
 		(stroke
@@
 	(wire
 		(pts
-			(xy 271.78 73.66) (xy 265.43 73.66)
+			(xy 102.87 33.02) (xy 102.87 31.75)
 		)
 		(stroke
@@
 	(wire
 		(pts
-			(xy 271.78 86.36) (xy 265.43 86.36)
-		)
-		(stroke
-			(width 0)
-			(type default)
-		)
-	)
-	(wire
-		(pts
 			(xy 247.65 71.12) (xy 252.73 71.12)
 		)
@@
 	(wire
 		(pts
+			(xy 265.43 73.66) (xy 271.78 73.66)
+		)
+		(stroke
+			(width 0)
+			(type default)
+		)
+	)
+	(wire
+		(pts
 			(xy 52.07 34.29) (xy 59.69 34.29)
 		)
@@
 	(wire
 		(pts
+			(xy 265.43 81.28) (xy 271.78 81.28)
+		)
+		(stroke
+			(width 0)
+			(type default)
+		)
+	)
+	(wire
+		(pts
 			(xy 36.83 120.65) (xy 36.83 127)
 		)
@@
 	(wire
 		(pts
+			(xy 265.43 76.2) (xy 271.78 76.2)
+		)
+		(stroke
+			(width 0)
+			(type default)
+		)
+	)
+	(wire
+		(pts
 			(xy 271.78 49.53) (xy 271.78 52.07)
 		)
@@
 	(wire
 		(pts
+			(xy 265.43 71.12) (xy 271.78 71.12)
+		)
+		(stroke
+			(width 0)
+			(type default)
+		)
+	)
+	(wire
+		(pts
 			(xy 176.53 139.7) (xy 179.07 139.7)
 		)
@@
 	(wire
 		(pts
-			(xy 271.78 71.12) (xy 265.43 71.12)
-		)
-		(stroke
-			(width 0)
-			(type default)
-		)
-	)
-	(wire
-		(pts
 			(xy 151.13 87.63) (xy 153.67 87.63)
 		)
@@
 	(wire
 		(pts
-			(xy 271.78 76.2) (xy 265.43 76.2)
-		)
-		(stroke
-			(width 0)
-			(type default)
-		)
-	)
-	(wire
-		(pts
 			(xy 275.59 127) (xy 275.59 129.54)
 		)
@@
 	(wire
 		(pts
+			(xy 265.43 86.36) (xy 271.78 86.36)
+		)
+		(stroke
+			(width 0)
+			(type default)
+		)
+	)
+	(wire
+		(pts
 			(xy 210.82 104.14) (xy 209.55 104.14)
 		)
@@
 	(wire
 		(pts
-			(xy 176.53 114.3) (xy 179.07 114.3)
+			(xy 265.43 78.74) (xy 271.78 78.74)
 		)
 		(stroke
@@
 	(wire
 		(pts
-			(xy 187.96 87.63) (xy 189.23 87.63)
+			(xy 176.53 114.3) (xy 179.07 114.3)
 		)
 		(stroke
@@
 	(wire
 		(pts
-			(xy 210.82 109.22) (xy 209.55 109.22)
+			(xy 187.96 87.63) (xy 189.23 87.63)
 		)
 		(stroke
@@
 	(wire
 		(pts
-			(xy 271.78 81.28) (xy 265.43 81.28)
+			(xy 210.82 109.22) (xy 209.55 109.22)
 		)
 		(stroke
@@
 	(wire
 		(pts
-			(xy 271.78 78.74) (xy 265.43 78.74)
-		)
-		(stroke
-			(width 0)
-			(type default)
-		)
-	)
-	(wire
-		(pts
 			(xy 48.26 34.29) (xy 52.07 34.29)
 		)
@@
 	(wire
 		(pts
-			(xy 271.78 83.82) (xy 265.43 83.82)
-		)
-		(stroke
-			(width 0)
-			(type default)
-		)
-	)
-	(wire
-		(pts
 			(xy 151.13 44.45) (xy 151.13 46.99)
 		)
@@
 	)
 	(symbol
-		(lib_id "Connector_Generic:Conn_02x10_Odd_Even")
-		(at 259.08 46.99 0)
-		(mirror y)
+		(lib_id "DF40C:DF40C-20DP-0.4V_51_")
+		(at 257.81 46.99 0)
 		(unit 1)
 		(exclude_from_sim no)
@@
 		(dnp no)
 		(property "Reference" "J7"
-			(at 257.81 30.48 0)
+			(at 259.08 30.48 0)
 			(effects
 				(font
@@
 		)
 		(property "Value" "Conn_02x10_Counter_Clockwise"
-			(at 257.81 33.02 0)
+			(at 259.08 33.02 0)
 			(effects
 				(font
@@
 			)
 		)
-		(property "Footprint" "Connector_Hirose_DF40:Hirose_DF40C-20DS-0.4V_2x10_P0.4mm"
-			(at 259.08 46.99 0)
+		(property "Footprint" "DF40C:HRS_DF40C-20DP-0.4V_51_"
+			(at 257.81 46.99 0)
 			(effects
 				(font
 					(size 1.27 1.27)
 				)
+				(justify bottom)
 				(hide yes)
 			)
 		)
 		(property "Datasheet" "~"
-			(at 259.08 46.99 0)
+			(at 257.81 46.99 0)
 			(effects
 				(font
@@
 		)
 		(property "Description" "Generic connector, double row, 02x10, odd/even pin numbering scheme (row 1 odd numbers, row 2 even numbers), script generated (kicad-library-utils/schlib/autogen/connector/)"
-			(at 259.08 46.99 0)
+			(at 257.81 46.99 0)
+			(effects
+				(font
+					(size 1.27 1.27)
+				)
+				(hide yes)
+			)
+		)
+		(property "PARTREV" "02/2020"
+			(at 257.81 46.99 0)
 			(effects
 				(font
 					(size 1.27 1.27)
 				)
+				(justify bottom)
+				(hide yes)
+			)
+		)
+		(property "STANDARD" "Manufacturer Recommendations"
+			(at 257.81 46.99 0)
+			(effects
+				(font
+					(size 1.27 1.27)
+				)
+				(justify bottom)
+				(hide yes)
+			)
+		)
+		(property "MAXIMUM_PACKAGE_HEIGHT" "1.29mm"
+			(at 257.81 46.99 0)
+			(effects
+				(font
+					(size 1.27 1.27)
+				)
+				(justify bottom)
+				(hide yes)
+			)
+		)
+		(property "MANUFACTURER" "Hirose Electric"
+			(at 257.81 46.99 0)
+			(effects
+				(font
+					(size 1.27 1.27)
+				)
+				(justify bottom)
 				(hide yes)
 			)
@@
 		)
 		(instances
-			(project "Controller base V0.5"
+			(project "Controller base V0.6"
 				(path "/5ff5287b-60c7-4258-8bdb-42f045207b2d"
 					(reference "J7")
@@
 			)
 		)
-		(property "Footprint" "Button_Switch_SMD:SW_SPST_PTS647_Sx38"
+		(property "Footprint" "Button_Switch_SMD:SW_Push_1P1T_XKB_TS-1187A"
 			(at 140.97 123.19 0)
 			(effects
@@
 	)
 	(symbol
-		(lib_id "Library:PRTR5V0U2X_215")
+		(lib_id "PRTR5V0U2X_215:PRTR5V0U2X_215")
 		(at 64.77 64.77 0)
 		(unit 1)
@@
 	)
 	(symbol
-		(lib_id "Connector_Generic:Conn_02x10_Odd_Even")
-		(at 260.35 81.28 0)
-		(mirror y)
+		(lib_id "DF40C:DF40C-20DP-0.4V_51_")
+		(at 259.08 81.28 0)
 		(unit 1)
 		(exclude_from_sim no)
@@
 		(dnp no)
 		(property "Reference" "J8"
-			(at 259.08 64.77 0)
+			(at 260.35 64.77 0)
 			(effects
 				(font
@@
 		)
 		(property "Value" "Conn_02x10_Counter_Clockwise"
-			(at 259.08 67.31 0)
+			(at 260.35 67.31 0)
 			(effects
 				(font
@@
 			)
 		)
-		(property "Footprint" "Connector_Hirose_DF40:Hirose_DF40C-20DS-0.4V_2x10_P0.4mm"
-			(at 260.35 81.28 0)
+		(property "Footprint" "DF40C:HRS_DF40C-20DP-0.4V_51_"
+			(at 259.08 81.28 0)
 			(effects
 				(font
 					(size 1.27 1.27)
 				)
+				(justify bottom)
 				(hide yes)
 			)
 		)
 		(property "Datasheet" "~"
-			(at 260.35 81.28 0)
+			(at 259.08 81.28 0)
 			(effects
 				(font
@@
 		)
 		(property "Description" "Generic connector, double row, 02x10, odd/even pin numbering scheme (row 1 odd numbers, row 2 even numbers), script generated (kicad-library-utils/schlib/autogen/connector/)"
-			(at 260.35 81.28 0)
+			(at 259.08 81.28 0)
 			(effects
 				(font
@@
 			)
 		)
+		(property "PARTREV" "02/2020"
+			(at 259.08 81.28 0)
+			(effects
+				(font
+					(size 1.27 1.27)
+				)
+				(justify bottom)
+				(hide yes)
+			)
+		)
+		(property "STANDARD" "Manufacturer Recommendations"
+			(at 259.08 81.28 0)
+			(effects
+				(font
+					(size 1.27 1.27)
+				)
+				(justify bottom)
+				(hide yes)
+			)
+		)
+		(property "MAXIMUM_PACKAGE_HEIGHT" "1.29mm"
+			(at 259.08 81.28 0)
+			(effects
+				(font
+					(size 1.27 1.27)
+				)
+				(justify bottom)
+				(hide yes)
+			)
+		)
+		(property "MANUFACTURER" "Hirose Electric"
+			(at 259.08 81.28 0)
+			(effects
+				(font
+					(size 1.27 1.27)
+				)
+				(justify bottom)
+				(hide yes)
+			)
+		)
 		(pin "19"
 		)
@@
 		)
 		(instances
-			(project "Controller base V0.5"
+			(project "Controller base V0.6"
 				(path "/5ff5287b-60c7-4258-8bdb-42f045207b2d"
 					(reference "J8")

Commit message: updated liby used
Parts:
- added TP1, TP2, TP3, TP4: TestPoint, MCU_Controller:TestPoint_Pad_D1.0mm, symbol Connector:TestPoint
- C1, C2, C3, C4, C5, C6, C7, C8: footprint Capacitor_SMD:C_0603_1608Metric_Pad1.08x0.95mm_HandSolder -> MCU_Controller:C_0603_1608Metric_Pad1.08x0.95mm_HandSolder; symbol Library:C -> MCU_Controller:C
- D1: footprint Diode_SMD:D_SOD-323 -> MCU_Controller:D_SOD-323; symbol Library:1N5819WS -> MCU_Controller:1N5819WS
- D2: footprint PRTR5V0U2X_215:PRTR5V0U2X_215 -> MCU_Controller:PRTR5V0U2X_215; symbol PRTR5V0U2X_215:PRTR5V0U2X_215 -> MCU_Controller:PRTR5V0U2X_215
- D3: footprint LED_SMD:LED_0603_1608Metric_Pad1.05x0.95mm_HandSolder -> MCU_Controller:LED_0603_1608Metric_Pad1.05x0.95mm_HandSolder; symbol Library:LED -> MCU_Controller:LED
- D4, D5, D6, D7: symbol Library:LED -> MCU_Controller:LED; now left out of the parts list
- J1: footprint 12402012E212A:USB_C_Receptacle_HRO_TYPE-C-31-M-12 -> MCU_Controller:USB_C_Receptacle_HRO_TYPE-C-31-M-12; symbol Library:USB_C_Receptacle_USB2.0_16P -> MCU_Controller:USB_C_Receptacle_USB2.0_16P
- J2: symbol Library:Conn_01x05_Pin -> MCU_Controller:Conn_01x05_Pin; now left out of the parts list
- J7, J8: footprint DF40C:HRS_DF40C-20DP-0.4V_51_ -> MCU_Controller:HRS_DF40C-20DP-0.4V_51_; symbol DF40C:DF40C-20DP-0.4V_51_ -> MCU_Controller:DF40C-20DP-0.4V_51_
- R1, R2, R3, R4, R5: footprint Resistor_SMD:R_0603_1608Metric_Pad0.98x0.95mm_HandSolder -> MCU_Controller:R_0603_1608Metric_Pad0.98x0.95mm_HandSolder; symbol Library:R -> MCU_Controller:R
- R10, R7, R8, R9: symbol Library:R -> MCU_Controller:R; now left out of the parts list
- R6: footprint Jumper:SolderJumper-2_P1.3mm_Open_RoundedPad1.0x1.5mm -> MCU_Controller:SolderJumper-2_P1.3mm_Open_RoundedPad1.0x1.5mm; symbol Library:R -> MCU_Controller:R
- SW1, SW2, SW3: symbol Library:SW_Push -> MCU_Controller:SW_Push; now left out of the parts list
- SW4: footprint Button_Switch_SMD:SW_Push_1P1T_XKB_TS-1187A -> MCU_Controller:SW_Push_1P1T_XKB_TS-1187A; symbol Library:SW_Push -> MCU_Controller:SW_Push
- U1: footprint AZ1117CH_3_3TRG1:SOT-223_DIO -> MCU_Controller:SOT-223_DIO; symbol Library:AZ1117CH-3.3TRG1 -> MCU_Controller:AZ1117CH-3.3TRG1
- U2: footprint PCM_Espressif:ESP32-S3-WROOM-1U -> MCU_Controller:ESP32-S3-WROOM-1U; symbol Library:ESP32-S3-WROOM-1 -> MCU_Controller:ESP32-S3-WROOM-1
Connections:
- net D+: now also TP4.1
- net D-: now also TP3.1
- net RXD0: now also TP1.1
- net TXD0: now also TP2.1

Commit message: generated bom
Parts:
- R6, TP1, TP2, TP3, TP4: now left out of the parts list
Changed lines of the file:
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@@
 		(unit 1)
 		(exclude_from_sim no)
-		(in_bom yes)
+		(in_bom no)
 		(on_board yes)
 		(dnp no)
@@
 		(unit 1)
 		(exclude_from_sim no)
-		(in_bom yes)
+		(in_bom no)
 		(on_board yes)
 		(dnp no)
@@
 		(unit 1)
 		(exclude_from_sim no)
-		(in_bom yes)
+		(in_bom no)
 		(on_board yes)
 		(dnp no)
@@
 		(unit 1)
 		(exclude_from_sim no)
-		(in_bom yes)
+		(in_bom no)
 		(on_board yes)
 		(dnp no)
@@
 		(unit 1)
 		(exclude_from_sim no)
-		(in_bom yes)
+		(in_bom no)
 		(on_board yes)
 		(dnp no)

Commit message: update
Parts:
- added H1, H2: MountingHole, MountingHole:MountingHole_2.5mm, symbol MCU_Controller:MountingHole
- TP1, TP2, TP3, TP4: symbol Connector:TestPoint -> MCU_Controller:TestPoint
Changed lines of the file:
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@@
 	)
 	(symbol
-		(lib_id "Connector:TestPoint")
+		(lib_id "MCU_Controller:TestPoint")
 		(at 81.28 59.69 0)
 		(unit 1)
@@
 	)
 	(symbol
-		(lib_id "Connector:TestPoint")
+		(lib_id "MCU_Controller:TestPoint")
 		(at 52.07 148.59 0)
 		(unit 1)
@@
 	)
 	(symbol
-		(lib_id "Connector:TestPoint")
+		(lib_id "MCU_Controller:TestPoint")
 		(at 73.66 44.45 0)
 		(unit 1)
@@
 	)
 	(symbol
+		(lib_id "MCU_Controller:MountingHole")
+		(at 86.36 109.22 0)
+		(unit 1)
+		(exclude_from_sim no)
+		(in_bom no)
+		(on_board yes)
+		(dnp no)
+		(property "Reference" "H1"
+			(at 88.9 107.9499 0)
+			(effects
+				(font
+					(size 1.27 1.27)
+				)
+				(justify left)
+			)
+		)
+		(property "Value" "MountingHole"
+			(at 79.756 112.268 0)
+			(effects
+				(font
+					(size 1.27 1.27)
+				)
+				(justify left)
+			)
+		)
+		(property "Footprint" "MountingHole:MountingHole_2.5mm"
+			(at 86.36 109.22 0)
+			(effects
+				(font
+					(size 1.27 1.27)
+				)
+				(hide yes)
+			)
+		)
+		(property "Datasheet" "~"
+			(at 86.36 109.22 0)
+			(effects
+				(font
+					(size 1.27 1.27)
+				)
+				(hide yes)
+			)
+		)
+		(property "Description" "Mounting Hole without connection"
+			(at 86.36 109.22 0)
+			(effects
+				(font
+					(size 1.27 1.27)
+				)
+				(hide yes)
+			)
+		)
+		(instances
+			(project ""
+				(path "/5ff5287b-60c7-4258-8bdb-42f045207b2d"
+					(reference "H1")
+					(unit 1)
+				)
+			)
+		)
+	)
+	(symbol
 		(lib_id "MCU_Controller:GND")
 		(at 269.24 154.94 0)
@@
 	)
 	(symbol
-		(lib_id "Connector:TestPoint")
+		(lib_id "MCU_Controller:TestPoint")
 		(at 63.5 149.86 0)
 		(unit 1)
@@
 					(unit 1)
 				)
+			)
+		)
+	)
+	(symbol
+		(lib_id "MCU_Controller:MountingHole")
+		(at 95.25 109.22 0)
+		(unit 1)
+		(exclude_from_sim no)
+		(in_bom no)
+		(on_board yes)
+		(dnp no)
+		(property "Reference" "H2"
+			(at 97.79 107.9499 0)
+			(effects
+				(font
+					(size 1.27 1.27)
+				)
+				(justify left)
+			)
+		)
+		(property "Value" "MountingHole"
+			(at 93.726 112.776 0)
+			(effects
+				(font
+					(size 1.27 1.27)
+				)
+				(justify left)
+			)
+		)
+		(property "Footprint" "MountingHole:MountingHole_2.5mm"
+			(at 95.25 109.22 0)
+			(effects
+				(font
+					(size 1.27 1.27)
+				)
+				(hide yes)
+			)
+		)
+		(property "Datasheet" "~"
+			(at 95.25 109.22 0)
+			(effects
+				(font
+					(size 1.27 1.27)
+				)
+				(hide yes)
+			)
+		)
+		(property "Description" "Mounting Hole without connection"
+			(at 95.25 109.22 0)
+			(effects
+				(font
+					(size 1.27 1.27)
+				)
+				(hide yes)
+			)
+		)
+		(instances
+			(project "Controller base V0.6"
+				(path "/5ff5287b-60c7-4258-8bdb-42f045207b2d"
+					(reference "H2")
+					(unit 1)
+				)

Commit message: slimed down files
Parts:
- removed D4, D5, D6, D7: LED, LED_SMD:LED_0603_1608Metric_Pad1.05x0.95mm_HandSolder, symbol MCU_Controller:LED
- removed R10, R7, R8, R9: 1K, Resistor_SMD:R_0603_1608Metric_Pad0.98x0.95mm_HandSolder, symbol MCU_Controller:R
- removed SW1, SW2, SW3: SW_Push, Button_Switch_SMD:SW_Push_1P1T_XKB_TS-1187A, symbol MCU_Controller:SW_Push
Other:
- removed sheet Input modules
- note removed: "Play Inicater LEDs"
- moved on the sheet: TP1, TP2, TP4
