File: Hardware/Controller/Controller.kicad_pcb (KiCad board)
At the start: 2 copper layers, 113.4 x 77.6 mm, 43 parts, among them J1 USB_C_Receptacle_USB2.0_16P, J2 Conn_01x05_Pin, SW1 SW_Push, SW10 SW_Push, SW11 SW_Push, SW12 SW_Push, SW13 SW_Push, SW14 SW_Push, SW15 SW_Push, SW16 SW_Push, SW2 SW_Push, SW3 SW_Push, SW4 SW_Push, SW5 SW_Push, SW6 SW_Push, SW7 SW_Push, SW8 SW_Push, SW9 SW_Push, U1 AZ1117CH-3.3TRG1, U2 ESP32-S3-WROOM-1U-N4, U3 COM-09032, U4 COM-09032

Commit message: update
Changed lines of the file:
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@@
 		(polygon
 			(pts
-				(xy 165.8 61.75) (xy 165.8 69.95) (xy 168.475 69.95) (xy 168.4 61.8)
+				(xy 162.5 60.101917) (xy 162.5 72.45) (xy 170.494326 72.45) (xy 170.382089 60.253496)
 			)
 		)

Commit message: current PCBs
Routing:
- net GND: track 36.4 -> 43.3 mm
Changed lines of the file:
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@@
 		)
+	)
+	(segment
+		(start 145.675 57.035)
+		(end 146.245 56.465)
+		(width 0.2)
+		(layer "F.Cu")
+		(net 1)
+	)
+	(segment
+		(start 145.675 58.45)
+		(end 145.675 60.075)
+		(width 0.2)
+		(layer "F.Cu")
+		(net 1)
+	)
+	(segment
+		(start 144.8 57.575)
+		(end 144.8 56.575)
+		(width 0.2)
+		(layer "F.Cu")
+		(net 1)
+	)
+	(segment
+		(start 145.675 58.45)
+		(end 145.675 57.035)
+		(width 0.2)
+		(layer "F.Cu")
+		(net 1)
+	)
+	(segment
+		(start 145.675 60.075)
+		(end 146.245 60.645)
+		(width 0.2)
+		(layer "F.Cu")
+		(net 1)
+	)
+	(segment
+		(start 145.675 58.45)
+		(end 144.8 57.575)
+		(width 0.2)
+		(layer "F.Cu")
+		(net 1)
 	)
 	(via
@@
 	)
 	(segment
+		(start 136.55 56.0575)
+		(end 136.55 61.7312)
+		(width 0.2)
+		(layer "F.Cu")
+		(net 20)
+	)
+	(segment
+		(start 137.2584 55.3491)
+		(end 136.55 56.0575)
+		(width 0.2)
+		(layer "F.Cu")
+		(net 20)
+	)
+	(segment
+		(start 171.9741 55.3491)
+		(end 137.2584 55.3491)
+		(width 0.2)
+		(layer "F.Cu")
+		(net 20)
+	)
+	(segment
+		(start 136.55 61.7312)
+		(end 137.2447 62.4259)
+		(width 0.2)
+		(layer "F.Cu")
+		(net 20)
+	)
+	(segment
 		(start 177.225 58.4)
 		(end 175.025 58.4)
@@
 	)
 	(segment
-		(start 136.7884 55.8191)
-		(end 136.7884 61.9696)
-		(width 0.2)
-		(layer "F.Cu")
-		(net 20)
-	)
-	(segment
-		(start 171.9741 55.3491)
-		(end 137.2584 55.3491)
-		(width 0.2)
-		(layer "F.Cu")
-		(net 20)
-	)
-	(segment
-		(start 136.7884 61.9696)
-		(end 137.2447 62.4259)
-		(width 0.2)
-		(layer "F.Cu")
-		(net 20)
-	)
-	(segment
 		(start 175.025 58.4)
 		(end 171.9741 55.3491)
@@
 		(net 20)
 	)
-	(segment
-		(start 137.2584 55.3491)
-		(end 136.7884 55.8191)
-		(width 0.2)
-		(layer "F.Cu")
-		(net 20)
-	)
 	(via
 		(at 137.2447 62.4259)
@@
 	)
 	(segment
-		(start 136.175 58.6)
+		(start 136.175 59.275)
 		(end 136.175 62.6392)
 		(width 0.2)
@@
 	)
 	(segment
+		(start 135.725 58.825)
+		(end 136.175 59.275)
+		(width 0.2)
+		(layer "F.Cu")
+		(net 23)
+	)
+	(segment
 		(start 157.6932 63.5046)
 		(end 171.85 63.5046)
@@
 	)
 	(via
-		(at 136.175 58.6)
+		(at 135.725 58.825)
 		(size 0.6)
 		(drill 0.3)
@@
 		(drill 0.3)
 		(layers "F.Cu" "B.Cu")
+		(net 23)
+	)
+	(segment
+		(start 148.4796 60.6103)
+		(end 148.4796 61.0251)
+		(width 0.2)
+		(layer "B.Cu")
+		(net 23)
+	)
+	(segment
+		(start 135.7585 58.7915)
+		(end 146.6608 58.7915)
+		(width 0.2)
+		(layer "B.Cu")
+		(net 23)
+	)
+	(segment
+		(start 135.8892 62.925)
+		(end 135.5517 62.925)
+		(width 0.2)
+		(layer "B.Cu")
+		(net 23)
+	)
+	(segment
+		(start 146.6608 58.7915)
+		(end 148.4796 60.6103)
+		(width 0.2)
+		(layer "B.Cu")
+		(net 23)
+	)
+	(segment
+		(start 174.9548 66.6094)
+		(end 174.9548 84.8048)
+		(width 0.2)
+		(layer "B.Cu")
+		(net 23)
+	)
+	(segment
+		(start 174.9548 84.8048)
+		(end 177.475 87.325)
+		(width 0.2)
+		(layer "B.Cu")
+		(net 23)
+	)
+	(segment
+		(start 171.85 63.5046)
+		(end 174.9548 66.6094)
+		(width 0.2)
+		(layer "B.Cu")
+		(net 23)
+	)
+	(segment
+		(start 135.725 58.825)
+		(end 135.7585 58.7915)
+		(width 0.2)
+		(layer "B.Cu")
 		(net 23)
 	)
@@
 	)
 	(segment
-		(start 135.8892 62.925)
-		(end 135.5517 62.925)
-		(width 0.2)
-		(layer "B.Cu")
-		(net 23)
-	)
-	(segment
-		(start 174.9548 66.6094)
-		(end 174.9548 84.8048)
-		(width 0.2)
-		(layer "B.Cu")
-		(net 23)
-	)
-	(segment
-		(start 174.9548 84.8048)
-		(end 177.475 87.325)
-		(width 0.2)
-		(layer "B.Cu")
-		(net 23)
-	)
-	(segment
-		(start 148.4796 60.6103)
-		(end 148.4796 61.0251)
-		(width 0.2)
-		(layer "B.Cu")
-		(net 23)
-	)
-	(segment
-		(start 171.85 63.5046)
-		(end 174.9548 66.6094)
-		(width 0.2)
-		(layer "B.Cu")
-		(net 23)
-	)
-	(segment
-		(start 136.46 58.6)
-		(end 136.6515 58.7915)
-		(width 0.2)
-		(layer "B.Cu")
-		(net 23)
-	)
-	(segment
-		(start 136.6515 58.7915)
-		(end 146.6608 58.7915)
-		(width 0.2)
-		(layer "B.Cu")
-		(net 23)
-	)
-	(segment
-		(start 136.175 58.6)
-		(end 136.46 58.6)
-		(width 0.2)
-		(layer "B.Cu")
-		(net 23)
-	)
-	(segment
 		(start 134.325 63.1)
 		(end 135.3767 63.1)
 		(width 0.2)
 		(layer "B.Cu")
-		(net 23)
-	)
-	(segment
-		(start 146.6608 58.7915)
-		(end 148.4796 60.6103)
-		(width 0.2)
-		(layer "B.Cu")
