File: Hardware/OSMC_Module_Buttons/OSMC_Module_Buttons.kicad_pcb (KiCad board)
At the start: 2 copper layers, 32 x 32 mm, 8 parts, among them J1 North Connector, J2 East Connector, J3 South Connector, J4 West Connector

Commit message: update
Parts:
- J1: value North Connector -> Right Arm
- J2: value East Connector -> Right Leg
- J3: value South Connector -> Left Leg
- J4: value West Connector -> Left Arm
Connections:
- J1 pad 4: unconnected-(J1-Pin_4-Pad4) -> GND
Routing:
- net Net-(J4-Pin_4): track 4.32 -> 11.7 mm
- net Net-(J4-Pin_2): track 19.4 -> 26.4 mm
- net Net-(J4-Pin_3): track 17.5 -> 24.3 mm
- net Net-(J4-Pin_1): track 11.4 -> 17.9 mm
Other:
- board text added: "Button V1 10/25"
- board text added: "Up"
