File: Hardware/OSMC_Module_Buttons/OSMC_Module_Buttons.kicad_sch (KiCad schematic)
At the start: 8 parts, among them J1 Right Arm, J2 Right Leg, J3 Left Leg, J4 Left Arm

Commit message: update
Connections:
- net GND: now also J1.4 (Pin_4)
- no-connect marks 0 -> 10
Changed lines of the file:
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@@
+	)
+	(junction
+		(at 160.02 111.76)
+		(diameter 0)
+		(color 0 0 0 0)
 	)
 	(junction
@@
 		(color 0 0 0 0)
 	)
+	(no_connect
+		(at 185.42 125.73)
+	)
+	(no_connect
+		(at 175.26 125.73)
+	)
+	(no_connect
+		(at 182.88 125.73)
+	)
+	(no_connect
+		(at 162.56 96.52)
+	)
+	(no_connect
+		(at 180.34 125.73)
+	)
+	(no_connect
+		(at 172.72 125.73)
+	)
+	(no_connect
+		(at 167.64 125.73)
+	)
+	(no_connect
+		(at 170.18 125.73)
+	)
+	(no_connect
+		(at 165.1 96.52)
+	)
+	(no_connect
+		(at 187.96 125.73)
+	)
 	(wire
 		(pts
@@
 	(wire
 		(pts
+			(xy 167.64 111.76) (xy 160.02 111.76)
+		)
+		(stroke
+			(width 0)
+			(type default)
+		)
+	)
+	(wire
+		(pts
 			(xy 149.86 96.52) (xy 149.86 99.06)
 		)
@@
 	(wire
 		(pts
-			(xy 134.62 113.03) (xy 134.62 111.76)
+			(xy 167.64 96.52) (xy 167.64 111.76)
+		)
+		(stroke
+			(width 0)
+			(type default)
+		)
+	)
+	(wire
+		(pts
+			(xy 134.62 114.3) (xy 134.62 111.76)
 		)
 		(stroke
@@
 	(symbol
 		(lib_id "power:GND")
-		(at 134.62 113.03 0)
+		(at 134.62 114.3 0)
 		(unit 1)
 		(exclude_from_sim no)
@@
 		(fields_autoplaced yes)
 		(property "Reference" "#PWR01"
+			(at 134.62 120.65 0)
+			(effects
+				(font
+					(size 1.27 1.27)
+				)
+				(hide yes)
+			)
+		)
+		(property "Value" "GND"
 			(at 134.62 119.38 0)
 			(effects
@@
 					(size 1.27 1.27)
 				)
-				(hide yes)
-			)
-		)
-		(property "Value" "GND"
-			(at 134.62 118.11 0)
-			(effects
-				(font
-					(size 1.27 1.27)
-				)
 			)
 		)
 		(property "Footprint" ""
-			(at 134.62 113.03 0)
+			(at 134.62 114.3 0)
 			(effects
 				(font
@@
 		)
 		(property "Datasheet" ""
-			(at 134.62 113.03 0)
+			(at 134.62 114.3 0)
 			(effects
 				(font
@@
 		)
 		(property "Description" "Power symbol creates a global label with name \"GND\" , ground"
-			(at 134.62 113.03 0)
-			(effects
-				(font
+			(at 134.62 114.3 0)
+			(effects
+				(font
