File: Hardware/OSMC_Module_Joystick/OSMC_Module_Joystick.kicad_pcb (KiCad board)
At the start: 2 copper layers, 32 x 32 mm, 5 parts, among them J1 Right Arm, J2 Right Leg, J3 Left Leg, J4 Left Arm, U1 COM-09032

Commit message: update
Connections:
- J1 pad 3: unconnected-(J1-Pin_3-Pad3) -> +5V
- J1 pad 4: unconnected-(J1-Pin_4-Pad4) -> GND
Routing:
- net +5V: track 40.6 -> 43.2 mm
Other:
- board text added: "Joystick V1 10/25"
- board text added: "Up"
