File: Hardware/OSMC_Module_Joystick/OSMC_Module_Joystick.kicad_sch (KiCad schematic)
At the start: 5 parts, among them J1 Right Arm, J2 Right Leg, J3 Left Leg, J4 Left Arm, U1 COM-09032

Commit message: update
Connections:
- net +5V: now also J1.3 (Pin_3)
- net GND: now also J1.4 (Pin_4)
- no-connect marks 0 -> 9
Changed lines of the file:
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@@
-	)
-	(junction
-		(at 125.73 116.84)
-		(diameter 0)
-		(color 0 0 0 0)
 	)
 	(junction
@@
 	)
 	(junction
-		(at 125.73 114.3)
-		(diameter 0)
-		(color 0 0 0 0)
-	)
-	(junction
-		(at 125.73 109.22)
-		(diameter 0)
-		(color 0 0 0 0)
-	)
-	(junction
-		(at 125.73 104.14)
+		(at 100.33 106.68)
+		(diameter 0)
+		(color 0 0 0 0)
+	)
+	(junction
+		(at 104.14 101.6)
 		(diameter 0)
 		(color 0 0 0 0)
@@
 	)
 	(junction
-		(at 125.73 111.76)
-		(diameter 0)
-		(color 0 0 0 0)
-	)
-	(junction
 		(at 120.65 109.22)
 		(diameter 0)
@@
 		(color 0 0 0 0)
 	)
+	(no_connect
+		(at 191.77 104.14)
+	)
+	(no_connect
+		(at 191.77 90.17)
+	)
+	(no_connect
+		(at 191.77 95.25)
+	)
+	(no_connect
+		(at 191.77 109.22)
+	)
+	(no_connect
+		(at 191.77 106.68)
+	)
+	(no_connect
+		(at 191.77 92.71)
+	)
+	(no_connect
+		(at 97.79 88.9)
+	)
+	(no_connect
+		(at 191.77 97.79)
+	)
+	(no_connect
+		(at 191.77 111.76)
+	)
+	(wire
+		(pts
+			(xy 104.14 101.6) (xy 104.14 104.14)
+		)
+		(stroke
+			(width 0)
+			(type default)
+		)
+	)
 	(wire
 		(pts
@@
 	(wire
 		(pts
+			(xy 97.79 101.6) (xy 104.14 101.6)
+		)
+		(stroke
+			(width 0)
+			(type default)
+		)
+	)
+	(wire
+		(pts
 			(xy 97.79 104.14) (xy 104.14 104.14)
 		)
@@
 	(wire
 		(pts
+			(xy 97.79 99.06) (xy 100.33 99.06)
+		)
+		(stroke
+			(width 0)
+			(type default)
+		)
+	)
+	(wire
+		(pts
 			(xy 123.19 83.82) (xy 125.73 83.82)
 		)
@@
 	(wire
 		(pts
-			(xy 128.27 116.84) (xy 125.73 116.84)
-		)
-		(stroke
-			(width 0)
-			(type default)
-		)
-	)
-	(wire
-		(pts
 			(xy 123.19 76.2) (xy 123.19 83.82)
 		)
@@
 	(wire
 		(pts
-			(xy 97.79 106.68) (xy 104.14 106.68)
+			(xy 97.79 106.68) (xy 100.33 106.68)
 		)
 		(stroke
@@
 	(wire
 		(pts
-			(xy 128.27 109.22) (xy 125.73 109.22)
-		)
-		(stroke
-			(width 0)
-			(type default)
-		)
-	)
-	(wire
-		(pts
 			(xy 125.73 91.44) (xy 118.11 91.44)
 		)
@@
 	(wire
 		(pts
+			(xy 100.33 106.68) (xy 104.14 106.68)
+		)
+		(stroke
+			(width 0)
+			(type default)
+		)
+	)
+	(wire
+		(pts
 			(xy 97.79 86.36) (xy 115.57 86.36)
 		)
@@
 	(wire
 		(pts
-			(xy 104.14 97.79) (xy 104.14 104.14)
+			(xy 104.14 97.79) (xy 104.14 101.6)
 		)
 		(stroke
@@
 	(wire
 		(pts
-			(xy 128.27 111.76) (xy 125.73 111.76)
-		)
-		(stroke
-			(width 0)
-			(type default)
-		)
-	)
-	(wire
-		(pts
-			(xy 128.27 114.3) (xy 125.73 114.3)
-		)
-		(stroke
-			(width 0)
-			(type default)
-		)
-	)
-	(wire
-		(pts
 			(xy 120.65 116.84) (xy 125.73 116.84)
 		)
@@
 	(wire
 		(pts
-			(xy 128.27 104.14) (xy 125.73 104.14)
-		)
-		(stroke
-			(width 0)
-			(type default)
-		)
-	)
-	(wire
-		(pts
 			(xy 123.19 93.98) (xy 123.19 83.82)
 		)
@@
 		)
 		(stroke
+			(width 0)
+			(type default)
+		)
+	)
+	(wire
+		(pts
+			(xy 100.33 99.06) (xy 100.33 106.68)
+		)
+		(stroke
