File: Hardware/MCU Carrier Board/MCU Carrier Board.kicad_sch (KiCad schematic)
At the start: 46 parts, among them J1 Conn_01x06_Pin, J2 Conn_01x06_Pin, J3 Conn_01x06_Pin, J4 Top Connector, J5 Bottom Connector, J6 Conn_01x06_Pin, J7 Conn_01x06_Pin, J8 Conn_01x06_Pin, J9 Conn_01x05_Pin, SW1 SW_Push, SW10 SW_Push, SW11 SW_Push, SW12 SW_Push, SW13 SW_Push, SW14 SW_Push, SW15 SW_Push, SW2 SW_Push, SW3 SW_Push, SW4 SW_Push, SW5 SW_Push, SW6 SW_Push, SW7 SW_Push, SW8 SW_Push, SW9 SW_Push, U1 Left Joystick, U2 Right Joystick

Commit message: update
Parts:
- removed C5, C6, C7, C8: 1uF, Capacitor_SMD:C_0603_1608Metric_Pad1.08x0.95mm_HandSolder, symbol Device:C
- removed SW1, SW10, SW11, SW12, SW13, SW14, SW15, SW2, SW6, SW7, SW8, SW9: SW_Push, Button_Switch_THT:SW_PUSH_6mm, symbol Switch:SW_Push
- removed U1: Left Joystick, COM_09032:XDCR_COM-09032, symbol COM-09032:Joystick-09032
- removed U2: Right Joystick, COM_09032:XDCR_COM-09032, symbol COM-09032:Joystick-09032
Connections:
- net GND: no longer J5.15, J5.17
- net GPIO39: now reaches J2.5 (Pin_5)
- net GPIO39: now also J5.15
- net GPIO40: now reaches J7.2 (Pin_2)
- net GPIO40: now also J5.17
- no-connect marks 2 -> 0

Commit message: added test points
Parts:
- added 3V3, Gnd1, VBUS1: TestPoint, TestPoint:TestPoint_Pad_D1.0mm, symbol MCU_Controller:TestPoint
Connections:
- net GND: now also Gnd1.1
- net VCC_3V3: now also 3V3.1
- net VCC_5V: now also VBUS1.1

Commit message: updated footprints
Parts:
- 3V3, Gnd1, VBUS1: footprint TestPoint:TestPoint_Pad_D1.0mm -> MCU_Carrier_Board:TestPoint_Pad_D1.0mm; symbol MCU_Controller:TestPoint -> MCU Carrier Board:TestPoint
- C1, C2, C3, C4: footprint Capacitor_SMD:C_0603_1608Metric_Pad1.08x0.95mm_HandSolder -> MCU_Carrier_Board:C_0603_1608Metric_Pad1.08x0.95mm_HandSolder; symbol Device:C -> MCU Carrier Board:C
- D1, D2, D3, D4: footprint LED_SMD:LED_0603_1608Metric_Pad1.05x0.95mm_HandSolder -> MCU_Carrier_Board:LED_0603_1608Metric_Pad1.05x0.95mm_HandSolder; symbol MCU_Controller:LED -> MCU Carrier Board:LED
- H1, H2, H3, H4: footprint MountingHole:MountingHole_2.5mm -> MCU_Carrier_Board:MountingHole_2.5mm; symbol Mechanical:MountingHole -> MCU Carrier Board:MountingHole
- J1, J2, J3, J6, J7, J8: footprint Connector_PinHeader_1.27mm:PinHeader_1x06_P1.27mm_Vertical -> MCU_Carrier_Board:PinHeader_1x06_P1.27mm_Vertical; symbol Connector:Conn_01x06_Pin -> MCU Carrier Board:Conn_01x06_Pin
- J4: footprint DF40C:HRS_DF40C-20DS-0.4V_51_ -> MCU_Carrier_Board:HRS_DF40C-20DS-0.4V_51_; symbol DF40C:DF40C-20DS-0.4V_51_ -> MCU Carrier Board:DF40C-20DS-0.4V_51_
- J5: footprint DF40C:HRS_DF40C-20DS-0.4V_51_ -> MCU_Carrier_Boardr:HRS_DF40C-20DS-0.4V_51_; symbol DF40C:DF40C-20DS-0.4V_51_ -> MCU Carrier Board:DF40C-20DS-0.4V_51_
- J9: footprint Connector_JST:JST_EH_S5B-EH_1x05_P2.50mm_Horizontal -> MCU_Carrier_Board:JST_EH_S5B-EH_1x05_P2.50mm_Horizontal; symbol MCU_Controller:Conn_01x05_Pin -> MCU Carrier Board:Conn_01x05_Pin
- R1, R2, R3, R4: footprint Resistor_SMD:R_0603_1608Metric_Pad0.98x0.95mm_HandSolder -> MCU_Carrier_Board:R_0603_1608Metric_Pad0.98x0.95mm_HandSolder; symbol MCU_Controller:R -> MCU Carrier Board:R
- SW3, SW4, SW5: footprint Button_Switch_SMD:SW_Push_1P1T_XKB_TS-1187A -> MCU_Carrier_Board:SW_Push_1P1T_XKB_TS-1187A; symbol MCU_Controller:SW_Push -> MCU Carrier Board:SW_Push
