File: Hardware/MCU Carrier Board V1.1/MCU Carrier Board V1.1.kicad_pcb (KiCad board)
At the start: 2 copper layers, 31.8 x 50.8 mm, 30 parts, among them J1 Conn_01x06_Pin, J2 Conn_01x06_Pin, J3 Conn_01x06_Pin, J4 Top Connector, J5 Bottom Connector, J6 Conn_01x06_Pin, J7 Conn_01x06_Pin, J8 Conn_01x06_Pin, SW3 SW_Push, SW4 SW_Push, SW5 SW_Push

Commit message: update traces
Routing:
- net GPIO9: track 20.0 -> 18.3 mm
- net GPIO3: track 18.7 -> 17.1 mm
- net GPIO5: track 13.8 -> 12.7 mm
- net GPIO8: track 17.2 -> 16.5 mm
