File: module/Modules/Modules.kicad_sch (KiCad schematic)
At the start: 47 parts, among them J1 JST SH, J10 JST SH, J2 Conn_01x04, J3 Conn_01x04, J4 Conn_01x04, J5 JST SH, J6 JST SH, J7 Conn_01x04, J8 Conn_01x04, J9 Conn_01x04, U1 COM-09032, U10 LTC4317, U11 XIAO-ESP32-S3-DIP, U2 OSMC Module Board w/pins, U3 24LC32, U4 OSMC Module Board, U5 OSMC Module Board w/pins, U6 OSMC Module Board, U7 24AA02-OT, U8 PCF8574DWR, U9 ADS1115IDGS

Commit message: update
Parts:
- added J11: JST SH, Connector_JST:JST_SH_BM04B-SRSS-TB_1x04-1MP_P1.00mm_Vertical, symbol OSMC_parts:Conn_01x04_MountingPin
- C1, C2, C3, C4: footprint OSMC_partsC_0603_1608Metric_Pad1.08x0.95mm_HandSolder -> OSMC_parts:C_0603_1608Metric_Pad1.08x0.95mm_HandSolder
- J1, J10, J5, J6: footprint OSMC_partsXDCR_COM-09032 -> OSMC_parts:XDCR_COM-09032
- J2, J3, J4, J7, J8, J9: footprint OSMC_partsJST_SH_SM04B-SRSS-TB_1x04-1MP_P1.00mm_Horizontal -> OSMC_parts:JST_SH_SM04B-SRSS-TB_1x04-1MP_P1.00mm_Horizontal
- JP1: footprint OSMC_partsPinSocket_1x04_P2.54mm_Vertical -> OSMC_parts:PinSocket_1x04_P2.54mm_Vertical
- JP2, R1, R2, R3, R4, R5, R6: footprint OSMC_partsSolderJumper-2_P1.3mm_Open_RoundedPad1.0x1.5mm -> OSMC_parts:SolderJumper-2_P1.3mm_Open_RoundedPad1.0x1.5mm
- R10, R11, R12, R13, R14, R15, R16, R17, R18, R19, R20, R7, R8, R9: footprint OSMC_partsModule standard large -> OSMC_parts:Module standard large
- U1: footprint OSMC_partsModule standard pin large -> OSMC_parts:Module standard pin large
- U10, U9: footprint OSMC_partsR_0805_2012Metric_Pad1.15x1.40mm_HandSolder -> OSMC_parts:R_0805_2012Metric_Pad1.15x1.40mm_HandSolder
- U11: footprint OSMC_partsXIAO-ESP32-S3-DIP -> OSMC_parts:XIAO-ESP32-S3-DIP
- U2: footprint OSMC_partsModule standard pin small -> OSMC_parts:Module standard pin small
- U3: footprint OSMC_partsModule standard small -> OSMC_parts:Module standard small
- U4: footprint OSMC_partsDFN-16-1EP_3x5mm_P0.5mm_EP1.66x4.4mm -> OSMC_parts:DFN-16-1EP_3x5mm_P0.5mm_EP1.66x4.4mm
- U5: footprint OSMC_partsSOIC-8_3.9x4.9mm_P1.27mm -> OSMC_parts:SOIC-8_3.9x4.9mm_P1.27mm
- U6: footprint OSMC_partsTSSOP-10_3x3mm_P0.5mm -> OSMC_parts:TSSOP-10_3x3mm_P0.5mm
- U7: footprint OSMC_partsSOT-23-5 -> OSMC_parts:SOT-23-5
- U8: footprint OSMC_partsDW16-L -> OSMC_parts:DW16-L
Connections:
- net Gnd: now also J11.1 (Pin_1)
- net SCL: now also J11.4 (Pin_4)
- net SDA: now also J11.3 (Pin_3)
- net Vdd: now also J11.2 (Pin_2)

Commit message: update
Parts:
- added J12: Conn_01x08_Socket, OSMC_parts:Button Spacing, symbol Connector:Conn_01x08_Socket
- added SW1: SW_Push, OSMC_parts:Membrane Button semi 4 mm, symbol Switch:SW_Push
- J1, J10, J5, J6: footprint OSMC_parts:XDCR_COM-09032 -> OSMC_parts:JST_SH_SM04B-SRSS-TB_1x04-1MP_P1.00mm_Horizontal
- J11: footprint Connector_JST:JST_SH_BM04B-SRSS-TB_1x04-1MP_P1.00mm_Vertical -> OSMC_parts:PinSocket_1x04_P2.54mm_Vertical
- J2, J3, J4, J7, J8, J9: footprint OSMC_parts:JST_SH_SM04B-SRSS-TB_1x04-1MP_P1.00mm_Horizontal -> Connector_JST:JST_SH_BM04B-SRSS-TB_1x04-1MP_P1.00mm_Vertical
- JP1: footprint OSMC_parts:PinSocket_1x04_P2.54mm_Vertical -> OSMC_parts:SolderJumper-2_P1.3mm_Open_RoundedPad1.0x1.5mm
- R1, R2, R3, R4, R5, R6: footprint OSMC_parts:SolderJumper-2_P1.3mm_Open_RoundedPad1.0x1.5mm -> OSMC_parts:R_0805_2012Metric_Pad1.15x1.40mm_HandSolder
- R10, R11, R12, R13, R14, R15, R16, R17, R18, R19, R20, R7, R8, R9: footprint OSMC_parts:Module standard large -> OSMC_parts:R_0805_2012Metric_Pad1.15x1.40mm_HandSolder
- U1: footprint OSMC_parts:Module standard pin large -> OSMC_parts:XDCR_COM-09032
- U10: footprint OSMC_parts:R_0805_2012Metric_Pad1.15x1.40mm_HandSolder -> OSMC_parts:TSSOP-10_3x3mm_P0.5mm
- U5: footprint OSMC_parts:SOIC-8_3.9x4.9mm_P1.27mm -> OSMC_parts:Module standard large
- U6: footprint OSMC_parts:TSSOP-10_3x3mm_P0.5mm -> OSMC_parts:Module standard pin large
- U9: footprint OSMC_parts:R_0805_2012Metric_Pad1.15x1.40mm_HandSolder -> OSMC_parts:SOIC-8_3.9x4.9mm_P1.27mm
Changed lines of the file:
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@@
 			)
 		)
-		(property "Footprint" "OSMC_parts:XDCR_COM-09032"
+		(property "Footprint" "OSMC_parts:JST_SH_SM04B-SRSS-TB_1x04-1MP_P1.00mm_Horizontal"
 			(at 189.23 156.21 0)
 			(effects
@@
 			)
 		)
-		(property "Footprint" "OSMC_parts:Module standard large"
+		(property "Footprint" "OSMC_parts:R_0805_2012Metric_Pad1.15x1.40mm_HandSolder"
 			(at 88.392 154.94 90)
 			(effects
@@
 			)
 		)
-		(property "Footprint" "OSMC_parts:JST_SH_SM04B-SRSS-TB_1x04-1MP_P1.00mm_Horizontal"
+		(property "Footprint" "Connector_JST:JST_SH_BM04B-SRSS-TB_1x04-1MP_P1.00mm_Vertical"
 			(at 203.2 156.21 0)
 			(effects
@@
 			)
 		)
-		(property "Footprint" "OSMC_parts:JST_SH_SM04B-SRSS-TB_1x04-1MP_P1.00mm_Horizontal"
+		(property "Footprint" "Connector_JST:JST_SH_BM04B-SRSS-TB_1x04-1MP_P1.00mm_Vertical"
 			(at 213.36 132.08 0)
 			(effects
@@
 			)
 		)
-		(property "Footprint" "OSMC_parts:SolderJumper-2_P1.3mm_Open_RoundedPad1.0x1.5mm"
+		(property "Footprint" "OSMC_parts:R_0805_2012Metric_Pad1.15x1.40mm_HandSolder"
 			(at 56.642 106.68 90)
 			(effects
@@
 			)
 		)
-		(property "Footprint" "OSMC_parts:PinSocket_1x04_P2.54mm_Vertical"
+		(property "Footprint" "OSMC_parts:SolderJumper-2_P1.3mm_Open_RoundedPad1.0x1.5mm"
 			(at 262.89 21.59 0)
 			(effects
@@
 			)
 		)
-		(property "Footprint" "OSMC_parts:Module standard large"
+		(property "Footprint" "OSMC_parts:R_0805_2012Metric_Pad1.15x1.40mm_HandSolder"
 			(at 189.992 59.69 90)
 			(effects
@@
 			)
 		)
-		(property "Footprint" "OSMC_parts:Module standard large"
+		(property "Footprint" "OSMC_parts:R_0805_2012Metric_Pad1.15x1.40mm_HandSolder"
 			(at 158.242 153.67 90)
 			(effects
@@
 			)
 		)
-		(property "Footprint" "OSMC_parts:XDCR_COM-09032"
+		(property "Footprint" "OSMC_parts:JST_SH_SM04B-SRSS-TB_1x04-1MP_P1.00mm_Horizontal"
 			(at 240.03 156.21 0)
 			(effects
@@
 			)
 		)
-		(property "Footprint" "OSMC_parts:JST_SH_SM04B-SRSS-TB_1x04-1MP_P1.00mm_Horizontal"
+		(property "Footprint" "Connector_JST:JST_SH_BM04B-SRSS-TB_1x04-1MP_P1.00mm_Vertical"
 			(at 257.81 156.21 0)
 			(effects
@@
 			)
 		)
-		(property "Footprint" "OSMC_parts:JST_SH_SM04B-SRSS-TB_1x04-1MP_P1.00mm_Horizontal"
+		(property "Footprint" "Connector_JST:JST_SH_BM04B-SRSS-TB_1x04-1MP_P1.00mm_Vertical"
 			(at 193.04 132.08 0)
 			(effects
@@
 			)
 		)
-		(property "Footprint" "OSMC_parts:SolderJumper-2_P1.3mm_Open_RoundedPad1.0x1.5mm"
+		(property "Footprint" "OSMC_parts:R_0805_2012Metric_Pad1.15x1.40mm_HandSolder"
 			(at 65.532 107.95 90)
 			(effects
@@
 			)
 		)
-		(property "Footprint" "OSMC_parts:Module standard large"
+		(property "Footprint" "OSMC_parts:R_0805_2012Metric_Pad1.15x1.40mm_HandSolder"
 			(at 112.522 90.17 90)
 			(effects
@@
 			)
 		)
-		(property "Footprint" "OSMC_parts:SolderJumper-2_P1.3mm_Open_RoundedPad1.0x1.5mm"
+		(property "Footprint" "OSMC_parts:R_0805_2012Metric_Pad1.15x1.40mm_HandSolder"
 			(at 74.422 109.22 90)
 			(effects
@@
 			)
 		)
-		(property "Footprint" "OSMC_parts:Module standard large"
+		(property "Footprint" "OSMC_parts:R_0805_2012Metric_Pad1.15x1.40mm_HandSolder"
 			(at 127.762 55.88 90)
 			(effects
@@
 			)
 		)
-		(property "Footprint" "OSMC_parts:Module standard large"
+		(property "Footprint" "OSMC_parts:R_0805_2012Metric_Pad1.15x1.40mm_HandSolder"
 			(at 182.372 59.69 90)
 			(effects
@@
 			)
 		)
-		(property "Footprint" "OSMC_parts:JST_SH_SM04B-SRSS-TB_1x04-1MP_P1.00mm_Horizontal"
+		(property "Footprint" "Connector_JST:JST_SH_BM04B-SRSS-TB_1x04-1MP_P1.00mm_Vertical"
 			(at 267.97 132.08 0)
 			(effects
@@
 			)
 		)
-		(property "Footprint" "OSMC_parts:R_0805_2012Metric_Pad1.15x1.40mm_HandSolder"
+		(property "Footprint" "OSMC_parts:SOIC-8_3.9x4.9mm_P1.27mm"
 			(at 77.47 48.26 0)
 			(effects
@@
 			)
 		)
-		(property "Footprint" "OSMC_parts:Module standard large"
+		(property "Footprint" "OSMC_parts:R_0805_2012Metric_Pad1.15x1.40mm_HandSolder"
 			(at 112.522 64.77 90)
 			(effects
@@
 			)
 		)
-		(property "Footprint" "OSMC_parts:XDCR_COM-09032"
+		(property "Footprint" "OSMC_parts:JST_SH_SM04B-SRSS-TB_1x04-1MP_P1.00mm_Horizontal"
 			(at 222.25 156.21 0)
 			(effects
@@
 	)
 	(symbol
+		(lib_id "Switch:SW_Push")
+		(at 157.48 130.81 0)
+		(unit 1)
+		(exclude_from_sim no)
+		(in_bom yes)
+		(on_board yes)
+		(dnp no)
+		(fields_autoplaced yes)
+		(property "Reference" "SW1"
+			(at 157.48 123.19 0)
+			(effects
+				(font
+					(size 1.27 1.27)
+				)
+			)
+		)
+		(property "Value" "SW_Push"
+			(at 157.48 125.73 0)
+			(effects
+				(font
+					(size 1.27 1.27)
+				)
+			)
+		)
+		(property "Footprint" "OSMC_parts:Membrane Button semi 4 mm"
+			(at 157.48 125.73 0)
+			(effects
+				(font
+					(size 1.27 1.27)
+				)
+				(hide yes)
+			)
+		)
+		(property "Datasheet" "~"
+			(at 157.48 125.73 0)
+			(effects
+				(font
+					(size 1.27 1.27)
+				)
+				(hide yes)
+			)
+		)
+		(property "Description" "Push button switch, generic, two pins"
+			(at 157.48 130.81 0)
+			(effects
+				(font
+					(size 1.27 1.27)
+				)
+				(hide yes)
+			)
+		)
+		(pin "1"
+		)
+		(pin "2"
+		)
+		(instances
+			(project ""
+				(path "/c7166619-b781-4a53-a071-e3ce369183d9"
+					(reference "SW1")
+					(unit 1)
+				)
+			)
+		)
+	)
+	(symbol
 		(lib_id "OSMC_parts:Input_Module")
 		(at 232.41 83.82 0)
@@
 			)
 		)
-		(property "Footprint" "OSMC_parts:SOIC-8_3.9x4.9mm_P1.27mm"
+		(property "Footprint" "OSMC_parts:Module standard large"
 			(at 232.41 83.82 0)
 			(effects
@@
 			)
 		)
-		(property "Footprint" "OSMC_parts:R_0805_2012Metric_Pad1.15x1.40mm_HandSolder"
+		(property "Footprint" "OSMC_parts:TSSOP-10_3x3mm_P0.5mm"
 			(at 152.4 101.6 0)
 			(effects
@@
 			)
 		)
-		(property "Footprint" "OSMC_parts:Module standard pin large"
+		(property "Footprint" "OSMC_parts:XDCR_COM-09032"
 			(at 45.72 44.45 0)
 			(effects
@@
 			)
 		)
-		(property "Footprint" "OSMC_parts:Module standard large"
+		(property "Footprint" "OSMC_parts:R_0805_2012Metric_Pad1.15x1.40mm_HandSolder"
 			(at 197.612 59.69 90)
 			(effects
@@
 	)
 	(symbol
+		(lib_id "Connector:Conn_01x08_Socket")
+		(at 171.45 119.38 0)
+		(unit 1)
+		(exclude_from_sim no)
+		(in_bom yes)
+		(on_board yes)
+		(dnp no)
+		(fields_autoplaced yes)
+		(property "Reference" "J12"
+			(at 172.72 119.3799 0)
+			(effects
+				(font
+					(size 1.27 1.27)
+				)
+				(justify left)
+			)
+		)
+		(property "Value" "Conn_01x08_Socket"
+			(at 172.72 121.9199 0)
+			(effects
+				(font
+					(size 1.27 1.27)
+				)
+				(justify left)
+			)
+		)
+		(property "Footprint" "OSMC_parts:Button Spacing"
+			(at 171.45 119.38 0)
+			(effects
+				(font
+					(size 1.27 1.27)
+				)
+				(hide yes)
+			)
+		)
+		(property "Datasheet" "~"
+			(at 171.45 119.38 0)
+			(effects
+				(font
+					(size 1.27 1.27)
+				)
+				(hide yes)
+			)
+		)
+		(property "Description" "Generic connector, single row, 01x08, script generated"
+			(at 171.45 119.38 0)
+			(effects
+				(font
+					(size 1.27 1.27)
+				)
+				(hide yes)
+			)
+		)
+		(pin "6"
+		)
+		(pin "1"
+		)
+		(pin "2"
+		)
+		(pin "4"
+		)
+		(pin "5"
+		)
+		(pin "3"
+		)
+		(pin "8"
+		)
+		(pin "7"
+		)
+		(instances
+			(project ""
+				(path "/c7166619-b781-4a53-a071-e3ce369183d9"
+					(reference "J12")
+					(unit 1)
+				)
+			)
+		)
+	)
+	(symbol
 		(lib_id "OSMC_parts:Input_Module_Pinless")
 		(at 264.16 82.55 0)
@@
 			)
 		)
-		(property "Footprint" "OSMC_parts:TSSOP-10_3x3mm_P0.5mm"
+		(property "Footprint" "OSMC_parts:Module standard pin large"
 			(at 264.16 82.55 0)
 			(effects
@@
 			)
 		)
-		(property "Footprint" "Connector_JST:JST_SH_BM04B-SRSS-TB_1x04-1MP_P1.00mm_Vertical"
+		(property "Footprint" "OSMC_parts:PinSocket_1x04_P2.54mm_Vertical"
 			(at 231.14 133.35 0)
 			(effects
@@
 			)
 		)
-		(property "Footprint" "OSMC_parts:SolderJumper-2_P1.3mm_Open_RoundedPad1.0x1.5mm"
+		(property "Footprint" "OSMC_parts:R_0805_2012Metric_Pad1.15x1.40mm_HandSolder"
 			(at 47.752 104.14 90)
 			(effects
@@
 			)
 		)
-		(property "Footprint" "OSMC_parts:JST_SH_SM04B-SRSS-TB_1x04-1MP_P1.00mm_Horizontal"
+		(property "Footprint" "Connector_JST:JST_SH_BM04B-SRSS-TB_1x04-1MP_P1.00mm_Vertical"
 			(at 247.65 132.08 0)
 			(effects
@@
 			)
 		)
-		(property "Footprint" "OSMC_parts:Module standard large"
+		(property "Footprint" "OSMC_parts:R_0805_2012Metric_Pad1.15x1.40mm_HandSolder"
 			(at 96.012 154.94 90)
 			(effects
@@
 			)
 		)
-		(property "Footprint" "OSMC_parts:SolderJumper-2_P1.3mm_Open_RoundedPad1.0x1.5mm"
+		(property "Footprint" "OSMC_parts:R_0805_2012Metric_Pad1.15x1.40mm_HandSolder"
 			(at 246.38 34.798 90)
 			(effects
@@
 			)
 		)
-		(property "Footprint" "OSMC_parts:Module standard large"
+		(property "Footprint" "OSMC_parts:R_0805_2012Metric_Pad1.15x1.40mm_HandSolder"
 			(at 174.752 59.69 90)
 			(effects
@@
 			)
 		)
-		(property "Footprint" "OSMC_parts:Module standard large"
+		(property "Footprint" "OSMC_parts:R_0805_2012Metric_Pad1.15x1.40mm_HandSolder"
 			(at 135.382 55.88 90)
 			(effects
@@
 			)
 		)
-		(property "Footprint" "OSMC_parts:Module standard large"
+		(property "Footprint" "OSMC_parts:R_0805_2012Metric_Pad1.15x1.40mm_HandSolder"
 			(at 121.412 90.17 90)
 			(effects
@@
 			)
 		)
-		(property "Footprint" "OSMC_parts:XDCR_COM-09032"
+		(property "Footprint" "OSMC_parts:JST_SH_SM04B-SRSS-TB_1x04-1MP_P1.00mm_Horizontal"
 			(at 276.86 156.21 0)
 			(effects
@@
 			)
 		)
-		(property "Footprint" "OSMC_parts:Module standard large"
+		(property "Footprint" "OSMC_parts:R_0805_2012Metric_Pad1.15x1.40mm_HandSolder"
 			(at 165.862 153.67 90)
 			(effects
@@
 			)
 		)
-		(property "Footprint" "OSMC_parts:Module standard large"
+		(property "Footprint" "OSMC_parts:R_0805_2012Metric_Pad1.15x1.40mm_HandSolder"
 			(at 121.412 64.77 90)
 			(effects
@@
 			)
 		)
-		(property "Footprint" "OSMC_parts:SolderJumper-2_P1.3mm_Open_RoundedPad1.0x1.5mm"
+		(property "Footprint" "OSMC_parts:R_0805_2012Metric_Pad1.15x1.40mm_HandSolder"
 			(at 246.38 23.368 90)
 			(effects

Commit message: update
Parts:
- added U12: MCP3428x-xSL, Package_SO:SOIC-14_3.9x8.7mm_P1.27mm, symbol Analog_ADC:MCP3428x-xSL
Changed lines of the file:
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@@
+	)
+	(symbol
+		(lib_id "Analog_ADC:MCP3428x-xSL")
+		(at 80.01 72.39 0)
+		(unit 1)
+		(exclude_from_sim no)
+		(in_bom yes)
+		(on_board yes)
+		(dnp no)
+		(fields_autoplaced yes)
+		(property "Reference" "U12"
+			(at 82.1533 57.15 0)
+			(effects
+				(font
+					(size 1.27 1.27)
+				)
+				(justify left)
+			)
+		)
+		(property "Value" "MCP3428x-xSL"
+			(at 82.1533 59.69 0)
+			(effects
+				(font
+					(size 1.27 1.27)
+				)
+				(justify left)
+			)
+		)
+		(property "Footprint" "Package_SO:SOIC-14_3.9x8.7mm_P1.27mm"
+			(at 101.6 86.36 0)
+			(effects
+				(font
+					(size 1.27 1.27)
+				)
+				(hide yes)
+			)
+		)
+		(property "Datasheet" "http://ww1.microchip.com/downloads/en/DeviceDoc/22226a.pdf"
+			(at 80.01 57.15 0)
+			(effects
+				(font
+					(size 1.27 1.27)
+				)
+				(hide yes)
+			)
+		)
+		(property "Description" "16-Bit, Multi-Channel ΔΣ Analog-to-Digital Converter with I2C Interface and On-Board Reference, SOIC-14"
+			(at 80.01 72.39 0)
+			(effects
+				(font
+					(size 1.27 1.27)
+				)
+				(hide yes)
+			)
+		)
+		(pin "2"
+		)
+		(pin "11"
+		)
+		(pin "12"
+		)
+		(pin "14"
+		)
+		(pin "3"
+		)
+		(pin "13"
+		)
+		(pin "10"
+		)
+		(pin "1"
+		)
+		(pin "4"
+		)
+		(pin "8"
+		)
+		(pin "5"
+		)
+		(pin "7"
+		)
+		(pin "9"
+		)
+		(pin "6"
+		)
+		(instances
+			(project ""
+				(path "/c7166619-b781-4a53-a071-e3ce369183d9"
+					(reference "U12")
+					(unit 1)
+				)
+			)
+		)
 	)
 	(symbol
