File: module/Navigation module/Navigation module.kicad_pcb (KiCad board)
At the start: 2 copper layers, 34 x 41 mm, 50 parts, among them J1 JST SH, J10 JST SH, J11 JST SH, J12 Conn_01x08_Socket, J2 Conn_01x04, J3 Conn_01x04, J4 Conn_01x04, J5 JST SH, J6 JST SH, J7 Conn_01x04, J8 Conn_01x04, J9 Conn_01x04, SW1 SW_Push, U1 COM-09032, U10 LTC4317, U11 XIAO-ESP32-S3-DIP, U12 MCP3428x-xSL, U2 OSMC Module Board w/pins, U4 OSMC Module Board, U5 OSMC Module Board w/pins, U6 OSMC Module Board, U7 24AA02-OT, U8 PCF8574DWR, U9 ADS1115IDGS

Commit message: update
Parts:
- removed U12: MCP3428x-xSL, Package_SO:SOIC-14_3.9x8.7mm_P1.27mm
- moved U1 122.3 mm to (168.6, 151.6)
