File: module/reciver board/Modules.kicad_sch (KiCad schematic)
At the start: 25 parts, among them U10 LTC4316xDD, U13 OSMC Module Board, U14 OSMC Module Board, U15 OSMC Module Board, U16 OSMC Module Board, U17 OSMC Module Board, U18 OSMC Module Board, U19 OSMC Module Board, U20 OSMC Module Board, U5 LTC4316xDD, U6 LTC4317

Commit message: update
Parts:
- removed U10, U5: LTC4316xDD, Package_DFN_QFN:DFN-10-1EP_3x3mm_P0.5mm_EP1.65x2.38mm, symbol Library:LTC4316xDD
- removed U13, U14, U15, U16, U17, U18, U19, U20: OSMC Module Board, OSMC_Module:Module standard large, symbol Library:Input_Module_Pinless
- added R19, R20, R21, R22, R23, R24, R29, R30, R31, R32, R33, R34, R39, R40, R41, R42, R43, R44: 10k, PCM_Resistor_SMD_AKL:R_0603_1608Metric_Pad1.05x0.95mm_HandSolder, symbol Library:R
- added R25, R26, R27, R28, R35, R36, R37, R38: R, PCM_Resistor_SMD_AKL:R_0603_1608Metric_Pad1.05x0.95mm_HandSolder, symbol Library:R
- added U2, U5, U7: LTC4317, Package_DFN_QFN:DFN-16-1EP_3x5mm_P0.5mm_EP1.66x4.4mm, symbol Library:LTC4317
- R10, R17, R18, R7, R8, R9: footprint PCM_Resistor_SMD_AKL:R_0805_2012Metric_Pad1.15x1.40mm_HandSolder -> PCM_Resistor_SMD_AKL:R_0603_1608Metric_Pad1.05x0.95mm_HandSolder
- R11, R12, R13, R14, R15, R16, R5, R6: value 10k -> R; footprint PCM_Resistor_SMD_AKL:R_0805_2012Metric_Pad1.15x1.40mm_HandSolder -> PCM_Resistor_SMD_AKL:R_0603_1608Metric_Pad1.05x0.95mm_HandSolder
Connections:
- net GND: now also R15.2, R17.1, R18.1, R6.2, U6.5 (XORH1), R19.1, R20.1, R26.2, R28.2, R29.1, R30.1, R36.2, R38.2, R39.1, R40.1, U2.1 (GND), U2.17 (EP), U2.3 (XORH2), U2.5 (XORH1), U5.1 (GND), U5.17 (EP), U5.3 (XORH2), U5.5 (XORH1), U7.1 (GND), U7.17 (EP), U7.3 (XORH2), U7.5 (XORH1); no longer U6.4 (XORL2)
- net P0: now also U2.10 (READY1), U5.10 (READY1), U7.10 (READY1)
- net P1: now also U2.9 (READY2), U5.9 (READY2), U7.9 (READY2)
- net SCL: now also U2.15 (SCLIN), U5.15 (SCLIN), U7.15 (SCLIN)
- net SCL0: no longer R5.2, R6.2, R8.2, U6.13 (SDAOUT1)
- net SCL1: no longer R10.2, U6.11 (SDAOUT2)
- net SDA: now also U2.12 (SDAIN), U5.12 (SDAIN), U7.12 (SDAIN)
- net VDD: now also R12.1, R21.1, R22.1, R23.1, R24.1, R25.1, R27.1, R31.1, R32.1, R33.1, R34.1, R35.1, R37.1, R41.1, R42.1, R43.1, R44.1, U2.7 (VCC), U5.7 (VCC), U7.7 (VCC); no longer R17.1, R18.1, R6.1
- net Det1: now reaches R17.2, U6.2 (ENABLE2)
- net at R11.2, R13.1: now also U6.4 (XORL2); no longer U6.5 (XORH1)
- net Det0: now reaches R18.2, U6.8 (ENABLE1)
- net at R15.1: now also R12.2, U2.4 (XORL2); no longer R12.1
- new net: R35.2, R36.1, R37.2, R38.1, U7.4 (XORL2), U7.6 (XORL1)
- new net: R25.2, R26.1, U5.6 (XORL1)
- new net: R5.2, R6.1, U2.6 (XORL1)
- new net: R27.2, R28.1, U5.4 (XORL2)
- new net Det2: R20.2, U2.8 (ENABLE1)
- new net Det3: R19.2, U2.2 (ENABLE2)
- new net Det4: R30.2, U5.8 (ENABLE1)
- new net Det5: R29.2, U5.2 (ENABLE2)
- new net Det6: R40.2, U7.8 (ENABLE1)
- new net Det7: R39.2, U7.2 (ENABLE2)
- new net SCL2: R21.2, U2.14 (SCLOUT1)
- new net SCL3: R23.2, U2.16 (SCLOUT2)
- new net SCL4: R31.2, U5.14 (SCLOUT1)
- new net SCL5: R33.2, U5.16 (SCLOUT2)
- new net SCL6: R41.2, U7.14 (SCLOUT1)
- new net SCL7: R43.2, U7.16 (SCLOUT2)
- new net SDA0: R8.2, U6.13 (SDAOUT1)
- new net SDA1: R10.2, U6.11 (SDAOUT2)
- new net SDA2: R22.2, U2.13 (SDAOUT1)
- new net SDA3: R24.2, U2.11 (SDAOUT2)
- new net SDA4: R32.2, U5.13 (SDAOUT1)
- new net SDA5: R34.2, U5.11 (SDAOUT2)
- new net SDA6: R42.2, U7.13 (SDAOUT1)
- new net SDA7: R44.2, U7.11 (SDAOUT2)
Other:
- added sheet Board attachment (attachment.kicad_sch)
- moved on the sheet: R10, R11, R13, R14, R16, R17, R18, R7, R8, R9, U6

Commit message: update
Parts:
- R11, R5: value R -> 976k
- R12, R6: value R -> 182k
- R13: value R -> 102k
- R15: value R -> 280k
- R16: value R -> 0
- R25, R27, R35, R37: value R -> 1000k
- R26: value R -> 392k
- R28: value R -> 523k
- R36: value R -> 681k
- R38: value R -> 887k
Connections:
- net at R35.2, R36.1, U7.6 (XORL1): no longer R37.2, R38.1, U7.4 (XORL2)
- new net: R37.2, R38.1, U7.4 (XORL2)
Changed lines of the file:
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@@
 	)
 	(junction
-		(at 215.9 125.73)
-		(diameter 0)
-		(color 0 0 0 0)
-	)
-	(junction
 		(at 78.74 92.71)
 		(diameter 0)
@@
 	)
 	(junction
-		(at 215.9 128.27)
-		(diameter 0)
-		(color 0 0 0 0)
-	)
-	(junction
 		(at 78.74 26.67)
 		(diameter 0)
@@
 	(wire
 		(pts
-			(xy 215.9 124.46) (xy 215.9 125.73)
-		)
-		(stroke
-			(width 0)
-			(type default)
-		)
-	)
-	(wire
-		(pts
 			(xy 210.82 53.34) (xy 210.82 71.12)
 		)
@@
 	(wire
 		(pts
+			(xy 228.6 138.43) (xy 231.14 138.43)
+		)
+		(stroke
+			(width 0)
+			(type default)
+		)
+	)
+	(wire
+		(pts
 			(xy 78.74 73.66) (xy 78.74 77.47)
 		)
@@
 	(wire
 		(pts
+			(xy 228.6 91.44) (xy 252.73 91.44)
+		)
+		(stroke
+			(width 0)
+			(type default)
+		)
+	)
+	(wire
+		(pts
 			(xy 118.11 96.52) (xy 125.73 96.52)
 		)
@@
 	(wire
 		(pts
-			(xy 215.9 128.27) (xy 182.88 128.27)
+			(xy 182.88 128.27) (xy 215.9 128.27)
 		)
 		(stroke
@@
 	(wire
 		(pts
-			(xy 228.6 91.44) (xy 252.73 91.44)
-		)
-		(stroke
-			(width 0)
-			(type default)
-		)
-	)
-	(wire
-		(pts
 			(xy 31.75 111.76) (xy 31.75 129.54)
 		)
@@
 	(wire
 		(pts
-			(xy 231.14 138.43) (xy 228.6 138.43)
-		)
-		(stroke
-			(width 0)
-			(type default)
-		)
-	)
-	(wire
-		(pts
 			(xy 17.78 157.48) (xy 24.13 157.48)
 		)
@@
 	(wire
 		(pts
-			(xy 215.9 125.73) (xy 215.9 128.27)
-		)
-		(stroke
-			(width 0)
-			(type default)
-		)
-	)
-	(wire
-		(pts
 			(xy 267.97 118.11) (xy 267.97 105.41)
 		)
@@
 	)
 	(label "SCL6"
-		(at 242.57 110.49 0)
+		(at 243.84 110.49 0)
 		(effects
 			(font
@@
 	)
 	(label "SDA6"
-		(at 242.57 113.03 0)
+		(at 243.84 113.03 0)
 		(effects
 			(font
@@
 			)
 		)
-		(property "Value" "R"
-			(at 168.91 107.95 0)
+		(property "Value" "1000k"
+			(at 166.878 107.696 0)
 			(effects
 				(font
@@
 			)
 		)
-		(property "Value" "R"
-			(at 26.67 108.966 0)
+		(property "Value" "182k"
+			(at 25.654 108.966 0)
 			(effects
 				(font
@@
 			)
 		)
-		(property "Value" "R"
+		(property "Value" "0"
 			(at 17.272 69.85 0)
 			(effects
@@
 			)
 		)
-		(property "Value" "R"
-			(at 27.178 134.62 0)
+		(property "Value" "280k"
+			(at 25.908 134.62 0)
 			(effects
 				(font
@@
 			)
 		)
-		(property "Value" "R"
+		(property "Value" "392k"
 			(at 165.862 67.31 0)
 			(effects
@@
 			)
 		)
-		(property "Value" "R"
+		(property "Value" "182k"
 			(at 17.272 135.89 0)
 			(effects
@@
 			)
 		)
-		(property "Value" "R"
-			(at 178.308 133.35 0)
+		(property "Value" "887k"
+			(at 176.784 133.604 0)
 			(effects
 				(font
@@
 			)
 		)
-		(property "Value" "R"
-			(at 175.26 40.386 0)
+		(property "Value" "1000k"
+			(at 173.228 39.878 0)
 			(effects
 				(font
@@
 			)
 		)
-		(property "Value" "R"
-			(at 175.768 66.04 0)
+		(property "Value" "523k"
+			(at 174.498 65.786 0)
 			(effects
 				(font
@@
 			)
 		)
-		(property "Value" "R"
-			(at 168.402 134.62 0)
+		(property "Value" "681k"
+			(at 167.894 134.112 0)
 			(effects
 				(font
@@
 			)
 		)
-		(property "Value" "R"
-			(at 17.78 109.22 0)
+		(property "Value" "976k"
+			(at 16.764 109.22 0)
 			(effects
 				(font
@@
 			)
 		)
-		(property "Value" "R"
-			(at 27.178 68.58 0)
+		(property "Value" "102k"
+			(at 25.908 68.58 0)
 			(effects
 				(font
@@
 			)
 		)
-		(property "Value" "R"
-			(at 166.37 40.64 0)
+		(property "Value" "1000k"
+			(at 164.338 40.132 0)
 			(effects
 				(font
@@
 			)
 		)
-		(property "Value" "R"
-			(at 26.67 42.926 0)
+		(property "Value" "976k"
+			(at 25.654 42.926 0)
 			(effects
 				(font
@@
 			)
 		)
-		(property "Value" "R"
-			(at 177.8 107.696 0)
+		(property "Value" "1000k"
+			(at 175.768 107.696 0)
 			(effects
 				(font

Commit message: started routing
Connections:
- net P0: no longer U2.10 (READY1), U5.10 (READY1), U7.10 (READY1)
- net P1: no longer U2.9 (READY2), U5.9 (READY2), U7.9 (READY2)
- net Det0 renamed EN0
- net Det1 renamed EN1
- net Det2 renamed EN2
- net Det3 renamed EN3
- net Det4 renamed EN4
- net Det5 renamed EN5
- net Det6 renamed EN6
- net Det7 renamed EN7
- new net P2: U2.10 (READY1)
- new net P3: U2.9 (READY2)
- new net P4: U5.10 (READY1)
- new net P5: U5.9 (READY2)
- new net P6: U7.10 (READY1)
- new net P7: U7.9 (READY2)
Other:
- sheet Board attachment ports: added Det0, Det1, Det2, Det3, Det4, Det5, Det6, Det7, SCL0, SCL1, SCL2, SCL3, SCL4, SCL5, SCL6, SCL7, SDA0, SDA1, SDA2, SDA3, SDA4, SDA5, SDA6, SDA7; removed none
