File: module/reciver board/attachment.kicad_sch (KiCad schematic)
At the start: 8 parts, among them U13 OSMC Module Board, U14 OSMC Module Board, U15 OSMC Module Board, U16 OSMC Module Board, U17 OSMC Module Board, U18 OSMC Module Board, U19 OSMC Module Board, U20 OSMC Module Board

Commit message: update
Parts:
- U13, U14, U15, U16, U17, U18, U19, U20: footprint OSMC_Module:Module standard large -> OSMC_Module:Module standard pin large outline; symbol Library:Input_Module_Pinless -> OSMC_Module:Input_Module
Connections:
- net Det0: now also U13.12 (Det), U13.13 (Det)
- net Det1: now also U15.12 (Det), U15.13 (Det)
- net Det2: now also U16.12 (Det), U16.13 (Det)
- net Det3: now also U18.12 (Det), U18.13 (Det)
- net Det4: now also U19.12 (Det), U19.13 (Det)
- net Det5: now also U17.12 (Det), U17.13 (Det)
- net Det6: now also U20.12 (Det), U20.13 (Det)
- net Det7: now also U14.12 (Det), U14.13 (Det)
- net SCL0: now also U13.4 (SCL), U13.8 (SCL)
- net SCL1: now also U15.4 (SCL), U15.8 (SCL)
- net SCL2: now also U16.4 (SCL), U16.8 (SCL)
- net SCL3: now also U18.4 (SCL), U18.8 (SCL)
- net SCL4: now also U17.3 (SDA), U17.7 (SDA)
- net SCL5: now also U20.4 (SCL), U20.8 (SCL)
- net SCL6: now also U14.4 (SCL), U14.8 (SCL)
- net SCL7: now also U19.4 (SCL), U19.8 (SCL)
- net SDA0: now also U13.3 (SDA), U13.7 (SDA)
- net SDA1: now also U15.3 (SDA), U15.7 (SDA)
- net SDA2: now also U16.3 (SDA), U16.7 (SDA)
- net SDA3: now also U18.3 (SDA), U18.7 (SDA)
- net SDA4: now also U17.4 (SCL), U17.8 (SCL)
- net SDA5: now also U20.3 (SDA), U20.7 (SDA)
- net SDA6: now also U14.3 (SDA), U14.7 (SDA)
- net SDA7: now also U19.3 (SDA), U19.7 (SDA)
- new net: U19.11 (OPT), U19.14 (OPT)
- new net: U17.11 (OPT), U17.14 (OPT)
- new net: U15.11 (OPT), U15.14 (OPT)
- new net: U18.11 (OPT), U18.14 (OPT)
- new net: U13.11 (OPT), U13.14 (OPT)
- new net: U20.11 (OPT), U20.14 (OPT)
- new net: U14.11 (OPT), U14.14 (OPT)
- new net: U16.11 (OPT), U16.14 (OPT)
- new net +5V: U13.10 (5V), U13.15 (5V), U14.10 (5V), U14.15 (5V), U15.10 (5V), U15.15 (5V), U16.10 (5V), U16.15 (5V), U17.10 (5V), U17.15 (5V), U18.10 (5V), U18.15 (5V), U19.10 (5V), U19.15 (5V), U20.10 (5V), U20.15 (5V)
- new net GND: U13.1 (Gnd), U13.16 (GND), U13.5 (Gnd), U13.9 (Gnd), U14.1 (Gnd), U14.16 (GND), U14.5 (Gnd), U14.9 (Gnd), U15.1 (Gnd), U15.16 (GND), U15.5 (Gnd), U15.9 (Gnd), U16.1 (Gnd), U16.16 (GND), U16.5 (Gnd), U16.9 (Gnd), U17.1 (Gnd), U17.16 (GND), U17.5 (Gnd), U17.9 (Gnd), U18.1 (Gnd), U18.16 (GND), U18.5 (Gnd), U18.9 (Gnd), U19.1 (Gnd), U19.16 (GND), U19.5 (Gnd), U19.9 (Gnd), U20.1 (Gnd), U20.16 (GND), U20.5 (Gnd), U20.9 (Gnd)
- new net VDD: U13.2 (Vdd), U13.6 (Vdd), U14.2 (Vdd), U14.6 (Vdd), U15.2 (Vdd), U15.6 (Vdd), U16.2 (Vdd), U16.6 (Vdd), U17.2 (Vdd), U17.6 (Vdd), U18.2 (Vdd), U18.6 (Vdd), U19.2 (Vdd), U19.6 (Vdd), U20.2 (Vdd), U20.6 (Vdd)
- no-connect marks 0 -> 40

Commit message: started routing
Connections:
- net Det4: now also U17.12 (Det), U17.13 (Det); no longer U19.12 (Det), U19.13 (Det)
- net Det5: now also U20.12 (Det), U20.13 (Det); no longer U17.12 (Det), U17.13 (Det)
- net Det6: now also U14.12 (Det), U14.13 (Det); no longer U20.12 (Det), U20.13 (Det)
- net Det7: now also U19.12 (Det), U19.13 (Det); no longer U14.12 (Det), U14.13 (Det)
Other:
- moved on the sheet: U14, U15, U16, U17, U18, U19, U20
