File: module/reciver board/reciver board.kicad_pcb (KiCad board)
At the start: 2 copper layers, 14 parts, among them U1 LTC4316xDD, U10 LTC4316xDD, U11 LTC4316xDD, U12 LTC4316xDD, U7 24AA02-OT, U9 LTC4316xDD

Commit message: update
Parts:
- removed R1: 100k, PCM_Resistor_SMD_AKL:R_0805_2012Metric_Pad1.15x1.40mm_HandSolder
- removed U11, U12, U9: LTC4316xDD, Package_DFN_QFN:DFN-10-1EP_3x3mm_P0.5mm_EP1.65x2.38mm
- removed U7: 24AA02-OT, Package_TO_SOT_SMD:SOT-23-5_HandSoldering
- added R10: 10k, PCM_Resistor_SMD_AKL:R_0805_2012Metric_Pad1.15x1.40mm_HandSolder, F.Cu at (98.0, 128.1)
- added R12: 10k, PCM_Resistor_SMD_AKL:R_0805_2012Metric_Pad1.15x1.40mm_HandSolder, F.Cu at (88.0, 111.7)
- added R15: 10k, PCM_Resistor_SMD_AKL:R_0805_2012Metric_Pad1.15x1.40mm_HandSolder, F.Cu at (88.0, 114.7)
- added R4: 100k, PCM_Resistor_SMD_AKL:R_0805_2012Metric_Pad1.15x1.40mm_HandSolder, F.Cu at (108.5, 151.7)
- added R5: 10k, PCM_Resistor_SMD_AKL:R_0805_2012Metric_Pad1.15x1.40mm_HandSolder, F.Cu at (88.0, 105.6)
- added R6: 10k, PCM_Resistor_SMD_AKL:R_0805_2012Metric_Pad1.15x1.40mm_HandSolder, F.Cu at (88.0, 108.7)
- added R7: 10k, PCM_Resistor_SMD_AKL:R_0805_2012Metric_Pad1.15x1.40mm_HandSolder, F.Cu at (98.0, 119.0)
- added R8: 10k, PCM_Resistor_SMD_AKL:R_0805_2012Metric_Pad1.15x1.40mm_HandSolder, F.Cu at (98.0, 122.0)
- added R9: 10k, PCM_Resistor_SMD_AKL:R_0805_2012Metric_Pad1.15x1.40mm_HandSolder, F.Cu at (98.0, 125.1)
- added U13: OSMC Module Board, OSMC_Module:Module standard large, F.Cu at (112.4, 80.0)
- added U14: OSMC Module Board, OSMC_Module:Module standard large, F.Cu at (155.4, 73.0)
- added U15: OSMC Module Board, OSMC_Module:Module standard large, F.Cu at (198.3, 80.2)
- added U16: OSMC Module Board, OSMC_Module:Module standard large, F.Cu at (181.4, 116.0)
- added U17: OSMC Module Board, OSMC_Module:Module standard large, B.Cu at (198.3, 80.2)
- added U18: OSMC Module Board, OSMC_Module:Module standard large, F.Cu at (129.4, 116.0)
- added U19: OSMC Module Board, OSMC_Module:Module standard large, B.Cu at (155.5, 123.0)
- added U20: OSMC Module Board, OSMC_Module:Module standard large, B.Cu at (112.4, 80.0)
- added U3: XIAO-ESP32-S3-DIP, Seed Studio Xiao:XIAO-ESP32-S3-DIP, B.Cu at (155.4, 67.7)
- added U4: PCF8574AT, PCF8574DWR:DW16-L, F.Cu at (156.1, 85.0)
- added U5: LTC4316xDD, Package_DFN_QFN:DFN-10-1EP_3x3mm_P0.5mm_EP1.65x2.38mm, B.Cu at (87.8, 125.8)
- added U6: LTC4317, Package_DFN_QFN:DFN-16-1EP_3x5mm_P0.5mm_EP1.66x4.4mm, F.Cu at (92.1, 123.7)
- C2: value 10 u -> .1 u
- JP1: value WP -> int
- JP2: value int -> WP
- U1: value LTC4316xDD -> 24AA02-OT; footprint Package_DFN_QFN:DFN-10-1EP_3x3mm_P0.5mm_EP1.65x2.38mm -> Package_TO_SOT_SMD:SOT-23-5
- moved U1 67.8 mm to (108.7, 155.6)
- moved R3 60.3 mm to (108.5, 148.7)
- moved C2 52.8 mm to (99.6, 151.0)
- moved C1 52.8 mm to (99.6, 148.4)
- moved C3 52.8 mm to (99.6, 153.5)
- moved C4 52.8 mm to (99.6, 156.0)
- moved JP1 52.8 mm to (103.9, 149.0)
- moved JP2 52.8 mm to (103.9, 152.5)
- moved U10 51.1 mm to (87.9, 122.6)
Connections:
- net /5V renamed +5V
- C1 pad 1: /Vdd -> VDD
- C1 pad 2: /Gnd -> GND
- C2 pad 1: /Vdd -> VDD
- C2 pad 2: /Gnd -> GND
- C3 pad 2: /Gnd -> GND
- C4 pad 2: /Gnd -> GND
- JP1 pad 1: /wp -> /int
- JP1 pad 2: /Vdd -> VDD
- JP2 pad 1: /int -> /wp
- JP2 pad 2: /Vdd -> VDD
- R3 pad 1: /Gnd -> GND
- U1 pad 1: unconnected-(U1-GND-Pad1) -> /SCL1
- U1 pad 2: unconnected-(U1-XORH-Pad2) -> GND
- U1 pad 3: unconnected-(U1-XORL-Pad3) -> /SDA1
- U1 pad 4: unconnected-(U1-V_{CC}-Pad4) -> VDD
- U1 pad 5: unconnected-(U1-ENABLE-Pad5) -> /wp
- U10 pad 4: unconnected-(U10-V_{CC}-Pad4) -> Net-(U10-V_{CC})
- U10 pad 8: unconnected-(U10-SDAOUT-Pad8) -> Net-(U10-SDAOUT)
- U10 pad 9: unconnected-(U10-SCLOUT-Pad9) -> Net-(U10-SCLOUT)
Other:
- board outline added: 41 x 34 mm

Commit message: update
Parts:
- removed U10: LTC4316xDD, Package_DFN_QFN:DFN-10-1EP_3x3mm_P0.5mm_EP1.65x2.38mm
- added R11: R, PCM_Resistor_SMD_AKL:R_0603_1608Metric_Pad1.05x0.95mm_HandSolder, F.Cu at (48.7, 91.5)
- added R13: R, PCM_Resistor_SMD_AKL:R_0603_1608Metric_Pad1.05x0.95mm_HandSolder, F.Cu at (48.7, 94.5)
- added R14: R, PCM_Resistor_SMD_AKL:R_0603_1608Metric_Pad1.05x0.95mm_HandSolder, F.Cu at (48.7, 97.6)
- added R16: R, PCM_Resistor_SMD_AKL:R_0603_1608Metric_Pad1.05x0.95mm_HandSolder, F.Cu at (48.7, 100.6)
- added R17: 10k, PCM_Resistor_SMD_AKL:R_0603_1608Metric_Pad1.05x0.95mm_HandSolder, F.Cu at (48.7, 103.6)
- added R18: 10k, PCM_Resistor_SMD_AKL:R_0603_1608Metric_Pad1.05x0.95mm_HandSolder, F.Cu at (48.7, 106.6)
- added R19: 10k, PCM_Resistor_SMD_AKL:R_0603_1608Metric_Pad1.05x0.95mm_HandSolder, F.Cu at (65.3, 77.0)
- added R20: 10k, PCM_Resistor_SMD_AKL:R_0603_1608Metric_Pad1.05x0.95mm_HandSolder, F.Cu at (67.8, 78.8)
- added R21: 10k, PCM_Resistor_SMD_AKL:R_0603_1608Metric_Pad1.05x0.95mm_HandSolder, F.Cu at (48.7, 115.7)
- added R22: 10k, PCM_Resistor_SMD_AKL:R_0603_1608Metric_Pad1.05x0.95mm_HandSolder, F.Cu at (53.5, 91.5)
- added R23: 10k, PCM_Resistor_SMD_AKL:R_0603_1608Metric_Pad1.05x0.95mm_HandSolder, F.Cu at (53.5, 94.5)
- added R24: 10k, PCM_Resistor_SMD_AKL:R_0603_1608Metric_Pad1.05x0.95mm_HandSolder, F.Cu at (53.5, 97.6)
- added R25: R, PCM_Resistor_SMD_AKL:R_0603_1608Metric_Pad1.05x0.95mm_HandSolder, F.Cu at (53.5, 100.6)
- added R26: R, PCM_Resistor_SMD_AKL:R_0603_1608Metric_Pad1.05x0.95mm_HandSolder, F.Cu at (53.5, 103.6)
- added R27: R, PCM_Resistor_SMD_AKL:R_0603_1608Metric_Pad1.05x0.95mm_HandSolder, F.Cu at (53.5, 106.6)
- added R28: R, PCM_Resistor_SMD_AKL:R_0603_1608Metric_Pad1.05x0.95mm_HandSolder, F.Cu at (53.5, 109.7)
- added R29: 10k, PCM_Resistor_SMD_AKL:R_0603_1608Metric_Pad1.05x0.95mm_HandSolder, F.Cu at (53.5, 112.7)
- added R30: 10k, PCM_Resistor_SMD_AKL:R_0603_1608Metric_Pad1.05x0.95mm_HandSolder, F.Cu at (53.5, 115.7)
- added R31: 10k, PCM_Resistor_SMD_AKL:R_0603_1608Metric_Pad1.05x0.95mm_HandSolder, F.Cu at (58.3, 91.5)
- added R32: 10k, PCM_Resistor_SMD_AKL:R_0603_1608Metric_Pad1.05x0.95mm_HandSolder, F.Cu at (58.3, 94.5)
- added R33: 10k, PCM_Resistor_SMD_AKL:R_0603_1608Metric_Pad1.05x0.95mm_HandSolder, F.Cu at (58.3, 97.6)
- added R34: 10k, PCM_Resistor_SMD_AKL:R_0603_1608Metric_Pad1.05x0.95mm_HandSolder, F.Cu at (58.3, 100.6)
- added R35: R, PCM_Resistor_SMD_AKL:R_0603_1608Metric_Pad1.05x0.95mm_HandSolder, F.Cu at (58.3, 103.6)
- added R36: R, PCM_Resistor_SMD_AKL:R_0603_1608Metric_Pad1.05x0.95mm_HandSolder, F.Cu at (58.3, 106.6)
- added R37: R, PCM_Resistor_SMD_AKL:R_0603_1608Metric_Pad1.05x0.95mm_HandSolder, F.Cu at (58.3, 109.7)
- added R38: R, PCM_Resistor_SMD_AKL:R_0603_1608Metric_Pad1.05x0.95mm_HandSolder, F.Cu at (58.3, 112.7)
- added R39: 10k, PCM_Resistor_SMD_AKL:R_0603_1608Metric_Pad1.05x0.95mm_HandSolder, F.Cu at (58.3, 115.7)
- added R40: 10k, PCM_Resistor_SMD_AKL:R_0603_1608Metric_Pad1.05x0.95mm_HandSolder, F.Cu at (63.1, 91.5)
- added R41: 10k, PCM_Resistor_SMD_AKL:R_0603_1608Metric_Pad1.05x0.95mm_HandSolder, F.Cu at (63.1, 94.5)
- added R42: 10k, PCM_Resistor_SMD_AKL:R_0603_1608Metric_Pad1.05x0.95mm_HandSolder, F.Cu at (63.1, 97.6)
- added R43: 10k, PCM_Resistor_SMD_AKL:R_0603_1608Metric_Pad1.05x0.95mm_HandSolder, F.Cu at (63.1, 100.6)
- added R44: 10k, PCM_Resistor_SMD_AKL:R_0603_1608Metric_Pad1.05x0.95mm_HandSolder, F.Cu at (63.1, 103.6)
- added U2: LTC4317, Package_DFN_QFN:DFN-16-1EP_3x5mm_P0.5mm_EP1.66x4.4mm, B.Cu at (176.0, 83.2)
- added U7: LTC4317, Package_DFN_QFN:DFN-16-1EP_3x5mm_P0.5mm_EP1.66x4.4mm, B.Cu at (136.3, 83.0)
- R10, R3, R4, R7, R8, R9: footprint PCM_Resistor_SMD_AKL:R_0805_2012Metric_Pad1.15x1.40mm_HandSolder -> PCM_Resistor_SMD_AKL:R_0603_1608Metric_Pad1.05x0.95mm_HandSolder
- R12, R15, R5, R6: value 10k -> R; footprint PCM_Resistor_SMD_AKL:R_0805_2012Metric_Pad1.15x1.40mm_HandSolder -> PCM_Resistor_SMD_AKL:R_0603_1608Metric_Pad1.05x0.95mm_HandSolder
- U4: value PCF8574AT -> PCF8574DWR
- U5: value LTC4316xDD -> LTC4317; footprint Package_DFN_QFN:DFN-10-1EP_3x3mm_P0.5mm_EP1.65x2.38mm -> Package_DFN_QFN:DFN-16-1EP_3x5mm_P0.5mm_EP1.66x4.4mm
- U6: moved to B.Cu
- moved U6 82.8 mm to (174.5, 116.0)
- moved U5 60.6 mm to (147.3, 114.3)
- moved U4 1.77 mm to (155.2, 83.5)
Connections:
- R10 pad 2: /Modules/SCL1 -> /Modules/SDA1
- R12 pad 1: Net-(U10-V_{CC}) -> VDD
- R12 pad 2: Net-(U10-SCLOUT) -> Net-(U2-XORL2)
- R15 pad 1: Net-(U10-V_{CC}) -> Net-(U2-XORL2)
- R15 pad 2: Net-(U10-SDAOUT) -> GND
- R5 pad 2: /Modules/SCL0 -> Net-(U2-XORL1)
- R6 pad 1: VDD -> Net-(U2-XORL1)
- R6 pad 2: /Modules/SCL0 -> GND
- R8 pad 2: /Modules/SCL0 -> /Modules/SDA0
- U5 pad 10: /Modules/SCLin -> /Modules/P0
- U5 pad 11: unconnected-(U5-EP-Pad11) -> /Modules/SDA5
- U5 pad 2: unconnected-(U5-XORH-Pad2) -> /Modules/EN5
- U5 pad 3: unconnected-(U5-XORL-Pad3) -> GND
- U5 pad 4: VDD -> Net-(U5-XORL2)
- U5 pad 5: unconnected-(U5-ENABLE-Pad5) -> GND
- U5 pad 6: unconnected-(U5-READY-Pad6) -> Net-(U5-XORL1)
- U5 pad 7: /Modules/SDAin -> VDD
- U5 pad 8: /Modules/SCL0 -> /Modules/EN4
- U5 pad 9: /Modules/SCL0 -> /Modules/P1
- U6 pad 10: unconnected-(U6-READY1-Pad10) -> /Modules/P0
- U6 pad 11: /Modules/SCL1 -> /Modules/SDA1
- U6 pad 13: /Modules/SCL0 -> /Modules/SDA0
- U6 pad 2: unconnected-(U6-ENABLE2-Pad2) -> /Modules/EN1
- U6 pad 3: unconnected-(U6-XORH2-Pad3) -> GND
- U6 pad 4: unconnected-(U6-XORL2-Pad4) -> Net-(U6-XORL2)
- U6 pad 5: unconnected-(U6-XORH1-Pad5) -> GND
- U6 pad 6: unconnected-(U6-XORL1-Pad6) -> Net-(U6-XORL1)
- U6 pad 8: unconnected-(U6-ENABLE1-Pad8) -> /Modules/EN0
- U6 pad 9: unconnected-(U6-READY2-Pad9) -> /Modules/P1

Commit message: update
Parts:
- added R1: 10k, PCM_Resistor_SMD_AKL:R_0603_1608Metric_Pad1.05x0.95mm_HandSolder, B.Cu at (167.9, 78.7)
- added R2: 10k, PCM_Resistor_SMD_AKL:R_0603_1608Metric_Pad1.05x0.95mm_HandSolder, B.Cu at (168.1, 74.4)
- added R45: 10k, PCM_Resistor_SMD_AKL:R_0603_1608Metric_Pad1.05x0.95mm_HandSolder, B.Cu at (144.2, 75.0)
- added R46: 10k, PCM_Resistor_SMD_AKL:R_0603_1608Metric_Pad1.05x0.95mm_HandSolder, B.Cu at (144.2, 78.7)
- C1, C2, C3, C4, JP1, JP2, R10, R14, R17, R18, R19, R20, R21, R22, R23, R24, R29, R3, R30, R31, R32, R33, R39, R4, R40, R41, R42, R43, R44, R7, R8, R9, U1: moved to B.Cu
- R11, R5: value R -> 976k; moved to B.Cu
- R12, R6: value R -> 182k; moved to B.Cu
- R13: value R -> 102k; moved to B.Cu
- R15: value R -> 280k; moved to B.Cu
- R16: value R -> 0; moved to B.Cu
- R25, R27, R35, R37: value R -> 1000k; moved to B.Cu
- R26: value R -> 392k; moved to B.Cu
- R28: value R -> 523k; moved to B.Cu
- R36: value R -> 681k; moved to B.Cu
- R38: value R -> 887k; moved to B.Cu
- U13, U14, U16, U18, U19, U20: footprint OSMC_Module:Module standard large -> OSMC_Module:Module standard pin large outline
- U15: footprint OSMC_Module:Module standard large -> OSMC_Module:Module standard pin large outline; moved to B.Cu
- U17: footprint OSMC_Module:Module standard large -> OSMC_Module:Module standard pin large outline; moved to F.Cu
- moved R18 136.8 mm to (185.3, 99.8), turned to -90 degrees
- moved R17 136.6 mm to (185.3, 104.6), turned to 90 degrees
- moved R11 134.3 mm to (182.3, 106.3), turned to 90 degrees
- moved R13 133.7 mm to (182.3, 101.8), turned to 90 degrees
- moved R14 130.6 mm to (179.0, 105.8), turned to 90 degrees
- moved R16 130.3 mm to (179.0, 100.9), turned to 90 degrees
- moved R22 108.3 mm to (159.9, 111.6), turned to 90 degrees
- moved R23 104.7 mm to (156.9, 111.6), turned to 90 degrees
- moved C4 104.1 mm to (140.2, 60.2), turned to -90 degrees
- moved R10 103.4 mm to (197.8, 100.8), turned to -90 degrees
- moved C3 102.8 mm to (143.0, 60.2), turned to -90 degrees
- moved R21 102.3 mm to (150.9, 111.6), turned to 90 degrees
- moved R24 101.3 mm to (153.9, 111.6), turned to 90 degrees
- moved R42 99.8 mm to (162.8, 103.7), turned to 90 degrees
- moved R7 98.7 mm to (195.6, 104.0), turned to 90 degrees
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Connections:
- JP1 pad 1: /int -> /INT
- R37 pad 2: Net-(U7-XORL1) -> Net-(U7-XORL2)
- R38 pad 1: Net-(U7-XORL1) -> Net-(U7-XORL2)
- R4 pad 2: /int -> /INT
- U7 pad 4: Net-(U7-XORL1) -> Net-(U7-XORL2)
Routing:
- added copper zone on In1.Cu, net GND
- added copper zone on In2.Cu, net VDD
Other:
- board size 41 x 34 mm -> 126.7 x 80.1 mm
- copper layers 2 -> 4

Commit message: started routing
Parts:
- R34: moved to B.Cu
- moved R25 48.6 mm to (106.8, 77.3), turned to -90 degrees
- moved R27 44.6 mm to (109.6, 78.2), turned to -90 degrees
- moved R34 44.0 mm to (124.0, 77.0), turned to -90 degrees
- moved R26 43.1 mm to (106.8, 82.0), turned to -90 degrees
- moved R28 40.0 mm to (109.6, 82.2), turned to -90 degrees
- moved R30 38.4 mm to (112.5, 75.8), turned to -90 degrees
- moved U5 37.6 mm to (115.9, 78.9)
- moved R32 37.5 mm to (121.0, 77.9)
- moved R33 37.5 mm to (120.3, 81.5)
- moved R6 37.1 mm to (185.5, 110.2), turned to 90 degrees
- moved R5 36.2 mm to (185.5, 114.9), turned to 90 degrees
- moved R29 35.8 mm to (112.5, 81.4), turned to 90 degrees
- moved R31 35.6 mm to (123.0, 80.5), turned to 90 degrees
- moved R14 34.0 mm to (202.8, 81.4)
- moved R16 33.8 mm to (202.8, 76.7)
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Connections:
- U13 pad 12: /Modules/Board attachment/Det0 -> /Modules/EN0
- U13 pad 13: /Modules/Board attachment/Det0 -> /Modules/EN0
- U13 pad 3: /Modules/Board attachment/SDA0 -> /Modules/SDA0
- U13 pad 4: /Modules/Board attachment/SCL0 -> /Modules/SCL0
- U13 pad 7: /Modules/Board attachment/SDA0 -> /Modules/SDA0
- U13 pad 8: /Modules/Board attachment/SCL0 -> /Modules/SCL0
- U14 pad 12: /Modules/Board attachment/Det7 -> /Modules/EN6
- U14 pad 13: /Modules/Board attachment/Det7 -> /Modules/EN6
- U14 pad 3: /Modules/Board attachment/SDA6 -> /Modules/SDA6
- U14 pad 4: /Modules/Board attachment/SCL6 -> /Modules/SCL6
- U14 pad 7: /Modules/Board attachment/SDA6 -> /Modules/SDA6
- U14 pad 8: /Modules/Board attachment/SCL6 -> /Modules/SCL6
- U15 pad 12: /Modules/Board attachment/Det1 -> /Modules/EN1
- U15 pad 13: /Modules/Board attachment/Det1 -> /Modules/EN1
- U15 pad 3: /Modules/Board attachment/SDA1 -> /Modules/SDA1
- U15 pad 4: /Modules/Board attachment/SCL1 -> /Modules/SCL1
- U15 pad 7: /Modules/Board attachment/SDA1 -> /Modules/SDA1
- U15 pad 8: /Modules/Board attachment/SCL1 -> /Modules/SCL1
- U16 pad 12: /Modules/Board attachment/Det2 -> /Modules/EN2
- U16 pad 13: /Modules/Board attachment/Det2 -> /Modules/EN2
- U16 pad 3: /Modules/Board attachment/SDA2 -> /Modules/SDA2
- U16 pad 4: /Modules/Board attachment/SCL2 -> /Modules/SCL2
- U16 pad 7: /Modules/Board attachment/SDA2 -> /Modules/SDA2
- U16 pad 8: /Modules/Board attachment/SCL2 -> /Modules/SCL2
- U17 pad 12: /Modules/Board attachment/Det5 -> /Modules/EN4
- U17 pad 13: /Modules/Board attachment/Det5 -> /Modules/EN4
- U17 pad 3: /Modules/Board attachment/SCL4 -> /Modules/SCL4
- U17 pad 4: /Modules/Board attachment/SDA4 -> /Modules/SDA4
- U17 pad 7: /Modules/Board attachment/SCL4 -> /Modules/SCL4
- U17 pad 8: /Modules/Board attachment/SDA4 -> /Modules/SDA4
- U18 pad 12: /Modules/Board attachment/Det3 -> /Modules/EN3
- U18 pad 13: /Modules/Board attachment/Det3 -> /Modules/EN3
- U18 pad 3: /Modules/Board attachment/SDA3 -> /Modules/SDA3
- U18 pad 4: /Modules/Board attachment/SCL3 -> /Modules/SCL3
- U18 pad 7: /Modules/Board attachment/SDA3 -> /Modules/SDA3
- U18 pad 8: /Modules/Board attachment/SCL3 -> /Modules/SCL3
- U19 pad 12: /Modules/Board attachment/Det4 -> /Modules/EN7
- U19 pad 13: /Modules/Board attachment/Det4 -> /Modules/EN7
- U19 pad 3: /Modules/Board attachment/SDA7 -> /Modules/SDA7
- U19 pad 4: /Modules/Board attachment/SCL7 -> /Modules/SCL7
- U19 pad 7: /Modules/Board attachment/SDA7 -> /Modules/SDA7
- U19 pad 8: /Modules/Board attachment/SCL7 -> /Modules/SCL7
- U2 pad 10: /Modules/P0 -> /Modules/P2
- U2 pad 12: /Modules/SDAin -> /SDA
- U2 pad 15: /Modules/SCLin -> /SCL
- U2 pad 9: /Modules/P1 -> /Modules/P3
- U20 pad 12: /Modules/Board attachment/Det6 -> /Modules/EN5
- U20 pad 13: /Modules/Board attachment/Det6 -> /Modules/EN5
- U20 pad 3: /Modules/Board attachment/SDA5 -> /Modules/SDA5
- U20 pad 4: /Modules/Board attachment/SCL5 -> /Modules/SCL5
- U20 pad 7: /Modules/Board attachment/SDA5 -> /Modules/SDA5
- U20 pad 8: /Modules/Board attachment/SCL5 -> /Modules/SCL5
- U4 pad 10: /P5 -> /Modules/P5
- U4 pad 11: /P6 -> /Modules/P6
- U4 pad 12: /P7 -> /Modules/P7
- U4 pad 4: /P0 -> /Modules/P0
- U4 pad 5: /P1 -> /Modules/P1
- U4 pad 6: /P2 -> /Modules/P2
- U4 pad 7: /P3 -> /Modules/P3
- U4 pad 9: /P4 -> /Modules/P4
- U5 pad 10: /Modules/P0 -> /Modules/P4
- U5 pad 12: /Modules/SDAin -> /SDA
- U5 pad 15: /Modules/SCLin -> /SCL
- U5 pad 9: /Modules/P1 -> /Modules/P5
- U6 pad 12: /Modules/SDAin -> /SDA
- U6 pad 15: /Modules/SCLin -> /SCL
- U7 pad 10: /Modules/P0 -> /Modules/P6
- U7 pad 12: /Modules/SDAin -> /SDA
- U7 pad 15: /Modules/SCLin -> /SCL
- U7 pad 9: /Modules/P1 -> /Modules/P7
Routing:
- net GND: track 0.00 -> 54.7 mm, vias 0 -> 8
- net /Modules/SDA7: track 0.00 -> 49.9 mm
- net /Modules/SCL6: track 0.00 -> 48.5 mm, vias 0 -> 1
- net /Modules/SDA6: track 0.00 -> 43.4 mm, vias 0 -> 1
- net /Modules/EN1: track 0.00 -> 42.7 mm, vias 0 -> 2
- net VDD: track 0.00 -> 40.6 mm, vias 0 -> 3
- net /Modules/SCL7: track 0.00 -> 34.5 mm
- net /Modules/SCL0: track 0.00 -> 30.1 mm, vias 0 -> 2
- net /Modules/SDA0: track 0.00 -> 29.6 mm, vias 0 -> 1
- net /Modules/SCL3: track 0.00 -> 26.9 mm, vias 0 -> 1
- net /Modules/SDA3: track 0.00 -> 26.8 mm, vias 0 -> 1
- net /Modules/SDA5: track 0.00 -> 19.3 mm
- net /Modules/SCL2: track 0.00 -> 18.2 mm, vias 0 -> 1
- net /Modules/SCL5: track 0.00 -> 18.1 mm
- net /Modules/EN5: track 0.00 -> 17.7 mm
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