File: module/OSMC_Module_Bumpers/OSMC_Module_Bumpers.kicad_sch (KiCad schematic)
At the start: 5 parts, among them SW1 SW_SPST, SW2 SW_SPST, U1 OSMC Module Board w/pins, U2 24LC02BT-I/OT, U3 PCF8574DWR

Commit message: reviewed PCBs
Parts:
- added JP1, JP2, JP3: SolderJumper_2_Bridged, Jumper:SolderJumper-2_P1.3mm_Bridged2Bar_Pad1.0x1.5mm, symbol Jumper:SolderJumper_2_Bridged
Connections:
- net 3v3: now also U3.16 (VCC)
- net 5V: no longer U3.16 (VCC)
- net GND: now also JP1.2 (B), JP2.2 (B), JP3.2 (B); no longer U3.1 (A0), U3.2 (A1), U3.3 (A2)
- net A2: now reaches U1.18 (A3)
- net A2: now also U3.3 (A2), JP3.1 (A)
- net A1: now reaches U1.19 (A2)
- net A1: now also U3.2 (A1), JP2.1 (A)
- net A0: now reaches U1.20 (A1)
- net A0: now also U3.1 (A0), JP1.1 (A)
- no-connect marks 10 -> 7
Other:
- moved on the sheet: SW1, SW2
