File: module/OSMC_Module_Generic_Receiver/OSMC_Module_Generic_Receiver.kicad_sch (KiCad schematic)
At the start: 1 part, among them U1 OSMC Module Board w/pins

Commit message: reviewed PCBs
Parts:
- added JP10, JP11, JP9: SolderJumper_3_Open, Jumper:SolderJumper-3_P1.3mm_Open_Pad1.0x1.5mm, symbol Jumper:SolderJumper_3_Open
Connections:
- net 3v3: now also JP10.1 (A), JP11.1 (A), JP9.1 (A); no longer U1.12 (Det), U1.13 (Int)
- net GND: now also JP10.3 (B), JP11.3 (B), JP9.3 (B)
- net at U1.18 (A3): now also JP9.2 (C)
- net at U1.19 (A2): now also JP10.2 (C)
- net at U1.20 (A1): now also JP11.2 (C)
- new net Det: U1.12 (Det), U1.13 (Int)
- no-connect marks 0 -> 1
Other:
- note added: "OSMC General Reciver Module"
- note removed: "OSMC Bumper Module"
