File: module/OSMC_Module_Generic_Receiver/OSMC_Module_Generic_Receiver.kicad_pcb (KiCad board)
At the start: 4 copper layers, 34 x 41 mm, 2 parts, among them U1 OSMC Module Board w/pins

Commit message: reviewed PCBs
Parts:
- added JP10: SolderJumper_3_Open, Jumper:SolderJumper-3_P1.3mm_Open_Pad1.0x1.5mm, F.Cu at (188.3, 68.9)
- added JP11: SolderJumper_3_Open, Jumper:SolderJumper-3_P1.3mm_Open_Pad1.0x1.5mm, F.Cu at (186.4, 70.7)
- added JP9: SolderJumper_3_Open, Jumper:SolderJumper-3_P1.3mm_Open_Pad1.0x1.5mm, F.Cu at (190.1, 67.0)
Connections:
- U1 pad 12: /3v3 -> /Det
- U1 pad 13: /3v3 -> /Det
- U1 pad 18: unconnected-(U1-A3-Pad18) -> Net-(JP9-C)
- U1 pad 19: unconnected-(U1-A2-Pad19) -> Net-(JP10-C)
- U1 pad 20: unconnected-(U1-A1-Pad20) -> Net-(JP11-C)
Routing:
- net /Det: track 0.00 -> 27.1 mm
- net /3v3: track 59.5 -> 46.0 mm, vias 2 -> 0
- net unconnected-(U1-PadMP)_3: track 12.4 -> 0.00 mm
- net GND: track 4.15 -> 8.17 mm, vias 2 -> 4
- net Net-(JP11-C): track 0.00 -> 3.40 mm
- net Net-(JP10-C): track 0.00 -> 3.37 mm
- net Net-(JP9-C): track 0.00 -> 3.36 mm
- net /SCL: track 18.6 -> 17.1 mm
- net /SDA: track 15.3 -> 16.0 mm
- net /INT: track 29.0 -> 28.5 mm
- added copper zone on B.Cu, net GND
- removed copper zone on In1.Cu, net GND
Other:
- board text added: "1 2 3"

Commit message: update to modules gerbers produced
Other:
- copper layers 4 -> 2
Changed lines of the file:
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@@
 	(layers
 		(0 "F.Cu" signal)
-		(4 "In1.Cu" signal)
-		(6 "In2.Cu" signal)
 		(2 "B.Cu" signal)
 		(9 "F.Adhes" user "F.Adhesive")
@@
 			)
 			(layer "dielectric 1"
-				(type "prepreg")
-				(thickness 0.1)
+				(type "core")
+				(thickness 1.51)
 				(material "FR4")
 				(epsilon_r 4.5)
-				(loss_tangent 0.02)
-			)
-			(layer "In1.Cu"
-				(type "copper")
-				(thickness 0.035)
-			)
-			(layer "dielectric 2"
-				(type "core")
-				(thickness 1.24)
-				(material "FR4")
-				(epsilon_r 4.5)
-				(loss_tangent 0.02)
-			)
-			(layer "In2.Cu"
-				(type "copper")
-				(thickness 0.035)
-			)
-			(layer "dielectric 3"
-				(type "prepreg")
-				(thickness 0.1)
-				(material "FR4")
-				(epsilon_r 4.5)

Commit message: created all gerber zips
Other:
- board text added: "GR MOD V1 2/26"
