File: module/OSMC_Module_Joystick/OSMC_Module_Joystick.kicad_sch (KiCad schematic)
At the start: 4 parts, among them U1 OSMC Module Board w/pins, U2 24LC02BT-I/OT, U3 ADS1115IDGS, U4 COM-09032

Commit message: reviewed PCBs
Parts:
- added JP1: SolderJumper_2_Bridged, Jumper:SolderJumper-2_P1.3mm_Bridged2Bar_RoundedPad1.0x1.5mm, symbol Jumper:SolderJumper_2_Bridged
- added R1: 100K, Resistor_SMD:R_0603_1608Metric_Pad0.98x0.95mm_HandSolder, symbol Device:R
Connections:
- net 3v3: now also R1.2
- net GND: now also U4.B2B (SEL-), JP1.1 (A); no longer U3.1 (ADDR)
- net A1: now reaches U1.20 (A1)
- net A1: now also U3.1 (ADDR), JP1.2 (B)
- net at U3.6 (AIN2), U4.B1A (SEL+): now also U4.B1B (SEL+), R1.1
- no-connect marks 0 -> 4
Changed lines of the file:
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@@
+	)
+	(junction
+		(at 101.6 156.21)
+		(diameter 0)
+		(color 0 0 0 0)
 	)
 	(junction
@@
 		(color 0 0 0 0)
 	)
+	(no_connect
+		(at 78.74 148.59)
+	)
+	(no_connect
+		(at 166.37 106.68)
+	)
+	(no_connect
+		(at 166.37 100.33)
+	)
+	(no_connect
+		(at 166.37 97.79)
+	)
 	(wire
 		(pts
@@
 	(wire
 		(pts
-			(xy 77.47 138.43) (xy 78.74 138.43)
+			(xy 78.74 133.35) (xy 78.74 138.43)
 		)
 		(stroke
@@
 	(wire
 		(pts
-			(xy 88.9 156.21) (xy 88.9 161.29)
+			(xy 88.9 156.21) (xy 88.9 167.64)
 		)
 		(stroke
@@
 	(wire
 		(pts
+			(xy 73.66 133.35) (xy 78.74 133.35)
+		)
+		(stroke
+			(width 0)
+			(type default)
+		)
+	)
+	(wire
+		(pts
 			(xy 129.54 76.2) (xy 134.62 76.2)
 		)
@@
 	(wire
 		(pts
+			(xy 161.29 102.87) (xy 166.37 102.87)
+		)
+		(stroke
+			(width 0)
+			(type default)
+		)
+	)
+	(wire
+		(pts
 			(xy 184.15 102.87) (xy 189.23 102.87)
 		)
@@
 	(wire
 		(pts
-			(xy 116.84 156.21) (xy 101.6 156.21)
+			(xy 101.6 156.21) (xy 116.84 156.21)
 		)
 		(stroke
@@
 	(wire
 		(pts
+			(xy 66.04 133.35) (xy 66.04 148.59)
+		)
+		(stroke
+			(width 0)
+			(type default)
+		)
+	)
+	(wire
+		(pts
 			(xy 111.76 140.97) (xy 111.76 151.13)
 		)
@@
 	(wire
 		(pts
+			(xy 101.6 167.64) (xy 101.6 166.37)
+		)
+		(stroke
+			(width 0)
+			(type default)
+		)
+	)
+	(wire
+		(pts
 			(xy 78.74 140.97) (xy 73.66 140.97)
 		)
@@
 	(wire
 		(pts
+			(xy 101.6 156.21) (xy 101.6 158.75)
+		)
+		(stroke
+			(width 0)
+			(type default)
+		)
+	)
+	(wire
+		(pts
 			(xy 116.84 146.05) (xy 99.06 146.05)
 		)
@@
 	(wire
 		(pts
-			(xy 77.47 137.16) (xy 77.47 138.43)
-		)
-		(stroke
-			(width 0)
-			(type default)
-		)
-	)
-	(wire
-		(pts
 			(xy 111.76 171.45) (xy 111.76 173.99)
 		)
@@
 		(pts
 			(xy 129.54 78.74) (xy 134.62 78.74)
+		)
+		(stroke
+			(width 0)
+			(type default)
+		)
+	)
+	(wire
+		(pts
+			(xy 101.6 167.64) (xy 88.9 167.64)
 		)
 		(stroke
@@
 		)
 	)
+	(label "A1"
+		(at 161.29 102.87 0)
+		(effects
+			(font
+				(size 1.27 1.27)
+			)
+			(justify left bottom)
+		)
+	)
 	(label "3v3"
 		(at 113.03 138.43 0)
@@
 		)
 	)
+	(label "A1"
+		(at 74.93 133.35 0)
+		(effects
+			(font
+				(size 1.27 1.27)
+			)
+			(justify left bottom)
+		)
+	)
 	(label "3v3"
-		(at 88.9 161.29 270)
+		(at 88.9 167.64 270)
 		(effects
 			(font
@@
 		(pin "V1"
 		)
+		(pin "B1B"
+		)
+		(pin "B2B"
+		)
 		(instances
 			(project ""
 				(path "/5710c097-548c-4b87-af5a-5a66621d409c"
 					(reference "U4")
+					(unit 1)
+				)
+			)
+		)
+	)
+	(symbol
+		(lib_id "Device:R")
+		(at 101.6 162.56 0)
+		(unit 1)
+		(exclude_from_sim no)
+		(in_bom yes)
+		(on_board yes)
+		(dnp no)
+		(fields_autoplaced yes)
+		(property "Reference" "R1"
+			(at 104.14 161.2899 0)
+			(effects
+				(font
+					(size 1.27 1.27)
+				)
+				(justify left)
+			)
+		)
+		(property "Value" "100K"
+			(at 104.14 163.8299 0)
+			(effects
+				(font
+					(size 1.27 1.27)
+				)
+				(justify left)
+			)
+		)
+		(property "Footprint" "Resistor_SMD:R_0603_1608Metric_Pad0.98x0.95mm_HandSolder"
+			(at 99.822 162.56 90)
+			(effects
+				(font
+					(size 1.27 1.27)
+				)
+				(hide yes)
+			)
+		)
+		(property "Datasheet" "~"
+			(at 101.6 162.56 0)
+			(effects
+				(font
+					(size 1.27 1.27)
+				)
+				(hide yes)
+			)
+		)
+		(property "Description" "Resistor"
+			(at 101.6 162.56 0)
+			(effects
+				(font
+					(size 1.27 1.27)
+				)
+				(hide yes)
+			)
+		)
+		(pin "1"
+		)
+		(pin "2"
+		)
+		(instances
+			(project ""
+				(path "/5710c097-548c-4b87-af5a-5a66621d409c"
+					(reference "R1")
 					(unit 1)
 				)
@@
 	)
 	(symbol
+		(lib_id "Jumper:SolderJumper_2_Bridged")
+		(at 69.85 133.35 0)
+		(unit 1)
+		(exclude_from_sim no)
+		(in_bom no)
+		(on_board yes)
+		(dnp no)
+		(fields_autoplaced yes)
+		(property "Reference" "JP1"
+			(at 69.85 127 0)
+			(effects
+				(font
+					(size 1.27 1.27)
+				)
+			)
+		)
+		(property "Value" "SolderJumper_2_Bridged"
+			(at 69.85 129.54 0)
+			(effects
+				(font
+					(size 1.27 1.27)
+				)
+			)
+		)
+		(property "Footprint" "Jumper:SolderJumper-2_P1.3mm_Bridged2Bar_RoundedPad1.0x1.5mm"
+			(at 69.85 133.35 0)
+			(effects
+				(font
+					(size 1.27 1.27)
+				)
+				(hide yes)
+			)
+		)
+		(property "Datasheet" "~"
+			(at 69.85 133.35 0)
+			(effects
+				(font
+					(size 1.27 1.27)
+				)
+				(hide yes)
+			)
+		)
+		(property "Description" "Solder Jumper, 2-pole, closed/bridged"
+			(at 69.85 133.35 0)
+			(effects
+				(font
+					(size 1.27 1.27)
+				)
+				(hide yes)
+			)
+		)
+		(pin "1"
+		)
+		(pin "2"
+		)
+		(instances
+			(project ""
+				(path "/5710c097-548c-4b87-af5a-5a66621d409c"
+					(reference "JP1")
+					(unit 1)
+				)
+			)
+		)
+	)
+	(symbol
 		(lib_id "power:GND")
 		(at 111.76 173.99 0)
@@
 	(symbol
 		(lib_id "power:GND")
-		(at 77.47 137.16 270)
+		(at 66.04 148.59 0)
 		(unit 1)
 		(exclude_from_sim no)
@@
 		(fields_autoplaced yes)
 		(property "Reference" "#PWR05"
-			(at 71.12 137.16 0)
+			(at 66.04 154.94 0)
 			(effects
 				(font
@@
 		)
 		(property "Value" "GND"
-			(at 73.66 137.1599 90)
-			(effects
-				(font
-					(size 1.27 1.27)
-				)
-				(justify right)
+			(at 68.58 149.8599 0)
+			(effects
+				(font
+					(size 1.27 1.27)
+				)
+				(justify left)
 			)
 		)
 		(property "Footprint" ""
-			(at 77.47 137.16 0)
+			(at 66.04 148.59 0)
 			(effects
 				(font
@@
 		)
 		(property "Datasheet" ""
-			(at 77.47 137.16 0)
+			(at 66.04 148.59 0)
 			(effects
 				(font
@@
 		)
 		(property "Description" "Power symbol creates a global label with name \"GND\" , ground"
-			(at 77.47 137.16 0)
-			(effects
-				(font
+			(at 66.04 148.59 0)
+			(effects
+				(font
