File: module/OSMC_Module_Joystick/OSMC_Module_Joystick.kicad_pcb (KiCad board)
At the start: 4 copper layers, 34 x 41 mm, 4 parts, among them U1 OSMC Module Board w/pins, U2 24LC02BT-I/OT, U3 ADS1115IDGS, U4 COM-09032

Commit message: reviewed PCBs
Parts:
- added JP1: SolderJumper_2_Bridged, Jumper:SolderJumper-2_P1.3mm_Bridged2Bar_RoundedPad1.0x1.5mm, B.Cu at (199.8, 71.5)
- added R1: 100K, Resistor_SMD:R_0603_1608Metric_Pad0.98x0.95mm_HandSolder, B.Cu at (197.1, 65.6)
- moved U2 2.38 mm to (197.1, 91.1)
Connections:
- U1 pad 20: unconnected-(U1-A1-Pad20) -> /A1
- U3 pad 1: GND -> /A1
- U4 pad B1B: (no net) -> Net-(U3-AIN2)
- U4 pad B2B: (no net) -> GND
Routing:
- net /3v3: track 102.2 -> 11.3 mm, vias 0 -> 4
- net GND: track 49.4 -> 15.4 mm, vias 0 -> 5
- net unconnected-(U1-PadMP)_3: track 29.4 -> 0.00 mm
- net /A1: track 0.00 -> 19.7 mm
- net /SDA: track 55.0 -> 38.5 mm, vias 2 -> 0
- net Net-(U3-AIN2): track 16.3 -> 24.5 mm, vias 0 -> 1
- net /SCL: track 49.6 -> 44.5 mm, vias 2 -> 0
- net Net-(U3-AIN1): track 13.4 -> 14.1 mm
- net Net-(U3-AIN0): track 14.1 -> 14.2 mm, vias 0 -> 1
- added copper zone on In2.Cu, net /3v3

Commit message: modules completed
Routing:
- net Net-(U3-AIN2): track 24.5 -> 27.4 mm
Changed lines of the file:
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@@
 	)
 	(segment
-		(start 195.53 74.64)
-		(end 193.43 76.74)
+		(start 195.53 64.705)
+		(end 193.865 63.04)
 		(width 0.2)
 		(layer "F.Cu")
@@
 	)
 	(segment
-		(start 195.53 64.705)
+		(start 193.6 76.57)
 		(end 195.53 74.64)
 		(width 0.2)
@@
 	)
 	(segment
-		(start 193.865 63.04)
+		(start 193.6 78.7)
+		(end 193.6 76.57)
+		(width 0.2)
+		(layer "F.Cu")
+		(net 16)
+	)
+	(segment
+		(start 195.53 74.64)
 		(end 195.53 64.705)
 		(width 0.2)
@@
 	)
 	(via
-		(at 193.43 76.74)
+		(at 193.6 78.7)
 		(size 0.6)
 		(drill 0.3)
 		(layers "F.Cu" "B.Cu")
+		(net 16)
+	)
+	(segment
+		(start 194.89 76.74)
+		(end 194.89 77.41)
+		(width 0.2)
+		(layer "B.Cu")
 		(net 16)
 	)
@@
 	)
 	(segment
-		(start 194.89 76.74)
-		(end 193.43 76.74)
+		(start 194.89 77.41)
+		(end 193.6 78.7)
 		(width 0.2)
 		(layer "B.Cu")

Commit message: created all gerber zips
Other:
- board text added: "J MOD V1 2/26"
