File: module/OSMC_Receiver/OSMC_Receiver.kicad_pcb (KiCad board)
At the start: 4 copper layers, 120.1 x 78.2 mm, 67 parts, among them U1 24AA02-OT, U13 OSMC Module Board, U14 OSMC Module Board, U15 OSMC Module Board, U16 OSMC Module Board, U17 OSMC Module Board, U18 OSMC Module Board, U19 OSMC Module Board, U2 LTC4317, U20 OSMC Module Board, U3 XIAO-ESP32-S3-DIP, U4 PCF8574DWR, U5 LTC4317, U6 LTC4317, U7 LTC4317

Commit message: reviewed PCBs
Parts:
- added JP10: SolderJumper_3_Open, Jumper:SolderJumper-3_P1.3mm_Open_Pad1.0x1.5mm, F.Cu at (205.2, 71.5)
- added JP11: SolderJumper_3_Open, Jumper:SolderJumper-3_P1.3mm_Open_Pad1.0x1.5mm, F.Cu at (203.3, 69.7)
- added JP12: SolderJumper_3_Open, Jumper:SolderJumper-3_P1.3mm_Open_Pad1.0x1.5mm, F.Cu at (119.2, 124.2)
- added JP13: SolderJumper_3_Open, Jumper:SolderJumper-3_P1.3mm_Open_Pad1.0x1.5mm, F.Cu at (121.0, 126.0)
- added JP14: SolderJumper_3_Open, Jumper:SolderJumper-3_P1.3mm_Open_Pad1.0x1.5mm, F.Cu at (122.9, 127.8)
- added JP15: SolderJumper_3_Open, Jumper:SolderJumper-3_P1.3mm_Open_Pad1.0x1.5mm, B.Cu at (148.5, 124.5)
- added JP16: SolderJumper_3_Open, Jumper:SolderJumper-3_P1.3mm_Open_Pad1.0x1.5mm, B.Cu at (146.6, 122.6)
- added JP17: SolderJumper_3_Open, Jumper:SolderJumper-3_P1.3mm_Open_Pad1.0x1.5mm, B.Cu at (144.8, 120.8)
- added JP18: SolderJumper_3_Open, Jumper:SolderJumper-3_P1.3mm_Open_Pad1.0x1.5mm, F.Cu at (103.5, 87.0)
- added JP19: SolderJumper_3_Open, Jumper:SolderJumper-3_P1.3mm_Open_Pad1.0x1.5mm, F.Cu at (105.3, 88.8)
- added JP20: SolderJumper_3_Open, Jumper:SolderJumper-3_P1.3mm_Open_Pad1.0x1.5mm, F.Cu at (107.2, 90.7)
- added JP21: SolderJumper_3_Open, Jumper:SolderJumper-3_P1.3mm_Open_Pad1.0x1.5mm, B.Cu at (103.7, 73.1)
- added JP22: SolderJumper_3_Open, Jumper:SolderJumper-3_P1.3mm_Open_Pad1.0x1.5mm, B.Cu at (105.5, 71.2)
- added JP23: SolderJumper_3_Open, Jumper:SolderJumper-3_P1.3mm_Open_Pad1.0x1.5mm, B.Cu at (107.4, 69.4)
- added JP24: SolderJumper_3_Open, Jumper:SolderJumper-3_P1.3mm_Open_Pad1.0x1.5mm, F.Cu at (143.9, 59.8)
- added JP25: SolderJumper_3_Open, Jumper:SolderJumper-3_P1.3mm_Open_Pad1.0x1.5mm, F.Cu at (142.1, 61.6)
- added JP26: SolderJumper_3_Open, Jumper:SolderJumper-3_P1.3mm_Open_Pad1.0x1.5mm, F.Cu at (140.3, 63.4)
- added JP3: SolderJumper_3_Open, Jumper:SolderJumper-3_P1.3mm_Open_Pad1.0x1.5mm, F.Cu at (191.7, 110.4)
- added JP4: SolderJumper_3_Open, Jumper:SolderJumper-3_P1.3mm_Open_Pad1.0x1.5mm, F.Cu at (189.8, 108.6)
- added JP5: SolderJumper_3_Open, Jumper:SolderJumper-3_P1.3mm_Open_Pad1.0x1.5mm, F.Cu at (188.0, 106.8)
- added JP6: SolderJumper_3_Open, Jumper:SolderJumper-3_P1.3mm_Open_Pad1.0x1.5mm, B.Cu at (207.1, 87.0)
- added JP7: SolderJumper_3_Open, Jumper:SolderJumper-3_P1.3mm_Open_Pad1.0x1.5mm, B.Cu at (205.3, 88.8)
- added JP8: SolderJumper_3_Open, Jumper:SolderJumper-3_P1.3mm_Open_Pad1.0x1.5mm, B.Cu at (203.4, 90.7)
- added JP9: SolderJumper_3_Open, Jumper:SolderJumper-3_P1.3mm_Open_Pad1.0x1.5mm, F.Cu at (207.0, 73.3)
Connections:
- U13 pad 18: unconnected-(U13-A3-Pad18) -> Net-(JP9-C)
- U13 pad 19: unconnected-(U13-A2-Pad19) -> Net-(JP10-C)
- U13 pad 20: unconnected-(U13-A1-Pad20) -> Net-(JP11-C)
- U14 pad 18: unconnected-(U14-A3-Pad18) -> Net-(JP24-C)
- U14 pad 19: unconnected-(U14-A2-Pad19) -> Net-(JP25-C)
- U14 pad 20: unconnected-(U14-A1-Pad20) -> Net-(JP26-C)
- U15 pad 18: unconnected-(U15-A3-Pad18) -> Net-(JP6-C)
- U15 pad 19: unconnected-(U15-A2-Pad19) -> Net-(JP7-C)
- U15 pad 20: unconnected-(U15-A1-Pad20) -> Net-(JP8-C)
- U16 pad 18: unconnected-(U16-A3-Pad18) -> Net-(JP3-C)
- U16 pad 19: unconnected-(U16-A2-Pad19) -> Net-(JP4-C)
- U16 pad 20: unconnected-(U16-A1-Pad20) -> Net-(JP5-C)
- U17 pad 18: unconnected-(U17-A3-Pad18) -> Net-(JP18-C)
- U17 pad 19: unconnected-(U17-A2-Pad19) -> Net-(JP19-C)
- U17 pad 20: unconnected-(U17-A1-Pad20) -> Net-(JP20-C)
- U18 pad 18: unconnected-(U18-A3-Pad18) -> Net-(JP12-C)
- U18 pad 19: unconnected-(U18-A2-Pad19) -> Net-(JP13-C)
- U18 pad 20: unconnected-(U18-A1-Pad20) -> Net-(JP14-C)
- U19 pad 18: unconnected-(U19-A3-Pad18) -> Net-(JP15-C)
- U19 pad 19: unconnected-(U19-A2-Pad19) -> Net-(JP16-C)
- U19 pad 20: unconnected-(U19-A1-Pad20) -> Net-(JP17-C)
- U20 pad 18: unconnected-(U20-A3-Pad18) -> Net-(JP21-C)
- U20 pad 19: unconnected-(U20-A2-Pad19) -> Net-(JP22-C)
- U20 pad 20: unconnected-(U20-A1-Pad20) -> Net-(JP23-C)
Routing:
- net GND: track 200.5 -> 274.6 mm, vias 54 -> 62
- net VDD: track 122.4 -> 178.1 mm, vias 34 -> 46
- net /Modules/EN5: track 46.9 -> 52.3 mm
- net Net-(JP9-C): track 0.00 -> 3.47 mm
- net Net-(JP11-C): track 0.00 -> 3.45 mm
- net Net-(JP6-C): track 0.00 -> 3.45 mm
- net Net-(JP10-C): track 0.00 -> 3.44 mm
- net Net-(JP3-C): track 0.00 -> 3.44 mm
- net Net-(JP7-C): track 0.00 -> 3.42 mm
- net Net-(JP4-C): track 0.00 -> 3.42 mm
- net Net-(JP23-C): track 0.00 -> 3.41 mm
- net Net-(JP8-C): track 0.00 -> 3.40 mm
- net Net-(JP5-C): track 0.00 -> 3.40 mm
- net Net-(JP17-C): track 0.00 -> 3.39 mm
- net Net-(JP22-C): track 0.00 -> 3.39 mm
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Other:
- board text added: "3 2 1"
