File: module/OSMC_Module_Buttons_Click/OSMC_Module_Buttons_Click.kicad_pcb (KiCad board)
At the start: 4 copper layers, 34 x 41 mm, 15 parts, among them J1 Conn_01x08_Socket, SW1 SW_Push, SW2 SW_Push, SW3 SW_Push, SW4 SW_Push, SW5 SW_Push, SW6 SW_Push, SW7 SW_Push, SW8 SW_Push, U1 OSMC Module Board w/pins, U2 24LC02BT-I/OT, U3 PCF8574DWR

Commit message: created all gerber zips
Routing:
- net GND: track 24.8 -> 17.5 mm, vias 9 -> 6
- net /B4: track 20.3 -> 21.0 mm
Other:
- board text added: "B MOD V1.1 2/26"
