File: module/OSMC_Module_Buttons_Membrane/OSMC_Module_Buttons_Membrane.kicad_pcb (KiCad board)
At the start: 4 copper layers, 34 x 41 mm, 7 parts, among them J1 Conn_01x08_Socket, J1 SolderJumper_2_Bridged, J2 SolderJumper_2_Bridged, J3 SolderJumper_2_Bridged, U1 OSMC Module Board w/pins, U2 24LC02BT-I/OT, U3 PCF8574DWR

Commit message: created all gerber zips
Other:
- board text added: "B MOD V1 2/26"
