File: module/OSMC_Receiver_Translators/Modules.kicad_sch (KiCad schematic)
At the start: 44 parts, among them U2 LTC4317, U5 LTC4317, U6 LTC4317, U7 LTC4317

Commit message: board update
Connections:
- no-connect marks 0 -> 8
Other:
- added sheet jst Connectors (jst_connection.kicad_sch)
