File: module/OSMC_Receiver_Translators/attachment.kicad_sch (KiCad schematic)
At the start: 8 parts, among them U13 OSMC Module Board, U14 OSMC Module Board, U15 OSMC Module Board, U16 OSMC Module Board, U17 OSMC Module Board, U18 OSMC Module Board, U19 OSMC Module Board, U20 OSMC Module Board

Commit message: board update
Connections:
- net SCL4: now also U17.4 (SCL), U17.8 (SCL); no longer U17.3 (SDA), U17.7 (SDA)
- net SDA4: now also U17.3 (SDA), U17.7 (SDA); no longer U17.4 (SCL), U17.8 (SCL)
Changed lines of the file:
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@@
+		)
+	)
+	(hierarchical_label "Det6"
+		(shape input)
+		(at 158.75 146.05 0)
+		(effects
+			(font
+				(size 1.27 1.27)
+			)
+			(justify left)
+		)
+	)
+	(hierarchical_label "SCL1"
+		(shape input)
+		(at 90.17 66.04 270)
+		(effects
+			(font
+				(size 1.27 1.27)
+			)
+			(justify right)
+		)
+	)
+	(hierarchical_label "SCL5"
+		(shape input)
+		(at 115.57 157.48 270)
+		(effects
+			(font
+				(size 1.27 1.27)
+			)
+			(justify right)
+		)
+	)
+	(hierarchical_label "Det2"
+		(shape input)
+		(at 161.29 53.34 0)
+		(effects
+			(font
+				(size 1.27 1.27)
+			)
+			(justify left)
+		)
+	)
+	(hierarchical_label "SCL0"
+		(shape input)
+		(at 27.94 64.77 270)
+		(effects
+			(font
+				(size 1.27 1.27)
+			)
+			(justify right)
+		)
+	)
+	(hierarchical_label "SDA6"
+		(shape input)
+		(at 146.05 157.48 270)
+		(effects
+			(font
+				(size 1.27 1.27)
+			)
+			(justify right)
+		)
+	)
+	(hierarchical_label "SDA1"
+		(shape input)
+		(at 87.63 66.04 270)
+		(effects
+			(font
+				(size 1.27 1.27)
+			)
+			(justify right)
+		)
+	)
+	(hierarchical_label "SCL7"
+		(shape input)
+		(at 52.07 157.48 270)
+		(effects
+			(font
+				(size 1.27 1.27)
+			)
+			(justify right)
+		)
+	)
+	(hierarchical_label "Det3"
+		(shape input)
+		(at 219.71 53.34 0)
+		(effects
+			(font
+				(size 1.27 1.27)
+			)
+			(justify left)
+		)
+	)
+	(hierarchical_label "Det0"
+		(shape input)
+		(at 39.37 53.34 0)
+		(effects
+			(font
+				(size 1.27 1.27)
+			)
+			(justify left)
+		)
+	)
+	(hierarchical_label "SDA4"
+		(shape input)
+		(at 81.28 157.48 270)
+		(effects
+			(font
+				(size 1.27 1.27)
+			)
+			(justify right)
+		)
+	)
+	(hierarchical_label "SCL2"
+		(shape input)
+		(at 149.86 59.69 270)
+		(effects
+			(font
+				(size 1.27 1.27)
+			)
+			(justify right)
+		)
+	)
+	(hierarchical_label "SCL6"
+		(shape input)
+		(at 148.59 157.48 270)
+		(effects
+			(font
+				(size 1.27 1.27)
+			)
+			(justify right)
+		)
+	)
+	(hierarchical_label "Det1"
+		(shape input)
+		(at 100.33 54.61 0)
+		(effects
+			(font
+				(size 1.27 1.27)
+			)
+			(justify left)
 		)
 	)
 	(hierarchical_label "SCL4"
 		(shape input)
-		(at 81.28 157.48 270)
-		(effects
-			(font
-				(size 1.27 1.27)
-			)
-			(justify right)
-		)
-	)
-	(hierarchical_label "Det6"
-		(shape input)
-		(at 158.75 146.05 0)
-		(effects
-			(font
-				(size 1.27 1.27)
-			)
-			(justify left)
-		)
-	)
-	(hierarchical_label "SCL1"
-		(shape input)
-		(at 90.17 66.04 270)
-		(effects
-			(font
-				(size 1.27 1.27)
-			)
-			(justify right)
-		)
-	)
-	(hierarchical_label "SCL5"
-		(shape input)
-		(at 115.57 157.48 270)
-		(effects
-			(font
-				(size 1.27 1.27)
-			)
-			(justify right)
-		)
-	)
-	(hierarchical_label "Det2"
-		(shape input)
-		(at 161.29 53.34 0)
-		(effects
-			(font
-				(size 1.27 1.27)
-			)
-			(justify left)
-		)
-	)
-	(hierarchical_label "SCL0"
-		(shape input)
-		(at 27.94 64.77 270)
-		(effects
-			(font
-				(size 1.27 1.27)
-			)
-			(justify right)
-		)
-	)
-	(hierarchical_label "SDA6"
-		(shape input)
-		(at 146.05 157.48 270)
-		(effects
-			(font
-				(size 1.27 1.27)
-			)
-			(justify right)
-		)
-	)
-	(hierarchical_label "SDA1"
-		(shape input)
-		(at 87.63 66.04 270)
-		(effects
-			(font
-				(size 1.27 1.27)
-			)
-			(justify right)
-		)
-	)
-	(hierarchical_label "SCL7"
-		(shape input)
-		(at 52.07 157.48 270)
-		(effects
-			(font
-				(size 1.27 1.27)
-			)
-			(justify right)
-		)
-	)
-	(hierarchical_label "Det3"
-		(shape input)
-		(at 219.71 53.34 0)
-		(effects
-			(font
-				(size 1.27 1.27)
-			)
-			(justify left)
-		)
-	)
-	(hierarchical_label "Det0"
-		(shape input)
-		(at 39.37 53.34 0)
-		(effects
-			(font
-				(size 1.27 1.27)
-			)
-			(justify left)
-		)
-	)
-	(hierarchical_label "SCL2"
-		(shape input)
-		(at 149.86 59.69 270)
-		(effects
-			(font
-				(size 1.27 1.27)
-			)
-			(justify right)
-		)
-	)
-	(hierarchical_label "SCL6"
-		(shape input)
-		(at 148.59 157.48 270)
-		(effects
-			(font
-				(size 1.27 1.27)
-			)
-			(justify right)
-		)
-	)
-	(hierarchical_label "Det1"
-		(shape input)
-		(at 100.33 54.61 0)
-		(effects
-			(font
-				(size 1.27 1.27)
-			)
-			(justify left)
+		(at 83.82 157.48 270)
+		(effects
+			(font
+				(size 1.27 1.27)
+			)
+			(justify right)
 		)
 	)
@@
 		(effects
 			(font
-				(size 1.27 1.27)
-			)
-			(justify right)
-		)
-	)
-	(hierarchical_label "SDA4"
-		(shape input)
-		(at 83.82 157.48 270)
-		(effects
-			(font
