File: module/OSMC_Receiver_V1.2/OSMC_Receiver_V1.2.kicad_pcb (KiCad board)
At the start: 4 copper layers, 120.7 x 78.7 mm, 99 parts, among them U1 24AA02-OT, U13 OSMC Module Board, U14 OSMC Module Board, U15 OSMC Module Board, U16 OSMC Module Board, U17 OSMC Module Board, U18 OSMC Module Board, U19 OSMC Module Board, U2 LTC4317, U20 OSMC Module Board, U3 XIAO-ESP32-S3-DIP, U4 PCF8574DWR, U5 LTC4317, U6 LTC4317, U7 LTC4317

Commit message: board update
Parts:
- added J1: Conn_01x04, OSMC_Module:CONN4_BM04B-SRSS_JST, F.Cu at (119.3, 31.0)
- added J10: Conn_01x04, OSMC_Module:CONN4_BM04B-SRSS_JST, F.Cu at (137.7, 36.9)
- added J11: Conn_01x04, OSMC_Module:CONN4_BM04B-SRSS_JST, F.Cu at (137.7, 42.9)
- added J12: Conn_01x04, OSMC_Module:CONN4_BM04B-SRSS_JST, F.Cu at (137.7, 48.9)
- added J13: Conn_01x04, OSMC_Module:CONN4_BM04B-SRSS_JST, F.Cu at (146.8, 31.0)
- added J14: Conn_01x04, OSMC_Module:CONN4_BM04B-SRSS_JST, F.Cu at (146.8, 36.9)
- added J15: Conn_01x04, OSMC_Module:CONN4_BM04B-SRSS_JST, F.Cu at (146.8, 42.9)
- added J16: Conn_01x04, OSMC_Module:CONN4_BM04B-SRSS_JST, F.Cu at (146.8, 48.9)
- added J2: Conn_01x04, OSMC_Module:CONN4_BM04B-SRSS_JST, F.Cu at (119.3, 36.9)
- added J3: Conn_01x04, OSMC_Module:CONN4_BM04B-SRSS_JST, F.Cu at (119.3, 42.9)
- added J4: Conn_01x04, OSMC_Module:CONN4_BM04B-SRSS_JST, F.Cu at (119.3, 48.9)
- added J5: Conn_01x04, OSMC_Module:CONN4_BM04B-SRSS_JST, F.Cu at (128.5, 31.0)
- added J6: Conn_01x04, OSMC_Module:CONN4_BM04B-SRSS_JST, F.Cu at (128.5, 36.9)
- added J7: Conn_01x04, OSMC_Module:CONN4_BM04B-SRSS_JST, F.Cu at (128.5, 42.9)
- added J8: Conn_01x04, OSMC_Module:CONN4_BM04B-SRSS_JST, F.Cu at (128.5, 48.9)
- added J9: Conn_01x04, OSMC_Module:CONN4_BM04B-SRSS_JST, F.Cu at (137.7, 31.0)
Connections:
- U13 pad 11: unconnected-(U13-OPT-Pad11)_1 -> /Modules/Board attachment/Opt0
- U13 pad 14: unconnected-(U13-OPT-Pad11) -> /Modules/Board attachment/Opt0
- U14 pad 11: unconnected-(U14-OPT-Pad11) -> /Modules/Board attachment/Opt6
- U14 pad 14: unconnected-(U14-OPT-Pad11)_1 -> /Modules/Board attachment/Opt6
- U15 pad 11: unconnected-(U15-OPT-Pad11) -> /Modules/Board attachment/Opt1
- U15 pad 14: unconnected-(U15-OPT-Pad11)_1 -> /Modules/Board attachment/Opt1
- U16 pad 11: unconnected-(U16-OPT-Pad11)_1 -> /Modules/Board attachment/Opt2
- U16 pad 14: unconnected-(U16-OPT-Pad11) -> /Modules/Board attachment/Opt2
- U17 pad 11: unconnected-(U17-OPT-Pad11) -> /Modules/Board attachment/Opt4
- U17 pad 14: unconnected-(U17-OPT-Pad11)_1 -> /Modules/Board attachment/Opt4
- U17 pad 3: /Modules/SCL4 -> /Modules/SDA4
- U17 pad 4: /Modules/SDA4 -> /Modules/SCL4
- U17 pad 7: /Modules/SCL4 -> /Modules/SDA4
- U17 pad 8: /Modules/SDA4 -> /Modules/SCL4
- U18 pad 11: unconnected-(U18-OPT-Pad11)_1 -> /Modules/Board attachment/Opt3
- U18 pad 14: unconnected-(U18-OPT-Pad11) -> /Modules/Board attachment/Opt3
- U19 pad 11: unconnected-(U19-OPT-Pad11) -> /Modules/Board attachment/Opt7
- U19 pad 14: unconnected-(U19-OPT-Pad11)_1 -> /Modules/Board attachment/Opt7
- U20 pad 11: unconnected-(U20-OPT-Pad11)_1 -> /Modules/Board attachment/Opt5
- U20 pad 14: unconnected-(U20-OPT-Pad11) -> /Modules/Board attachment/Opt5
Routing:
- net /Modules/SCL4: track 37.7 -> 36.6 mm
