File: module/OSMC_Receiver_V1.2/attachment.kicad_sch (KiCad schematic)
At the start: 32 parts, among them U13 OSMC Module Board, U14 OSMC Module Board, U15 OSMC Module Board, U16 OSMC Module Board, U17 OSMC Module Board, U18 OSMC Module Board, U19 OSMC Module Board, U20 OSMC Module Board

Commit message: board update
Connections:
- net SCL4: now also U17.4 (SCL), U17.8 (SCL); no longer U17.3 (SDA), U17.7 (SDA)
- net SDA4: now also U17.3 (SDA), U17.7 (SDA); no longer U17.4 (SCL), U17.8 (SCL)
- net Opt7: now reaches U19.11 (OPT), U19.14 (OPT)
- net Opt4: now reaches U17.11 (OPT), U17.14 (OPT)
- net Opt1: now reaches U15.11 (OPT), U15.14 (OPT)
- net Opt3: now reaches U18.11 (OPT), U18.14 (OPT)
- net Opt0: now reaches U13.11 (OPT), U13.14 (OPT)
- net Opt5: now reaches U20.11 (OPT), U20.14 (OPT)
- net Opt6: now reaches U14.11 (OPT), U14.14 (OPT)
- net Opt2: now reaches U16.11 (OPT), U16.14 (OPT)
- no-connect marks 16 -> 8
Other:
- added sheet jst connections (jst_connection.kicad_sch)
